Commit message: Prep for purge... old files gotta go

File: cori_ws/install/cori_description/share/cori_description/urdf/cori_bot.urdf.xacro (robot description, xacro)
@@ -1,416 +1 @@
-<?xml version="1.0"?>
-<robot name="cori_bot" xmlns:xacro="http://ros.org/wiki/xacro">
-  <!-- Global material definitions -->
-  <material name="white">
-    <color rgba="1 1 1 1"/>
-  </material>
-  <material name="grey">
-    <color rgba="0.5 0.5 0.5 1"/>
-  </material>
-  <material name="black">
-    <color rgba="0 0 0 1"/>
-  </material>
-  <!-- Macro for arm structure -->
-  <xacro:macro name="arm" params="side">
-    <link name="${side}_upper_arm">
-      <visual>
-        <geometry><box size="0.08 0.08 0.3"/></geometry>
-        <material name="black"/>
-      </visual>
-      <collision>
-        <geometry><box size="0.08 0.08 0.3"/></geometry>
-      </collision>
-      <inertial>
-        <mass value="1.0"/>
-        <inertia ixx="0.005" ixy="0" ixz="0" iyy="0.005" iyz="0" izz="0.002"/>
-      </inertial>
-    </link>
-    <gazebo reference="${side}_upper_arm">
-      <material>black</material>
-      <mu1>0.9</mu1>
-      <mu2>0.9</mu2>
-    </gazebo>
-    <xacro:property name="arm_offset_x" value="${side == 'left' ? 0.2 : -0.2}" />
-    <joint name="torso_to_${side}_upper_arm" type="revolute">
-      <parent link="torso"/>
-      <child link="${side}_upper_arm"/>
-      <origin xyz="${arm_offset_x} 0 0.35"/>
-      <axis xyz="0 1 0"/>
-      <limit lower="-1.57" upper="1.57" effort="10.0" velocity="1.0"/>
-      <transmission name="torso_to_${side}_upper_arm_trans">
-        <type>transmission_interface/SimpleTransmission</type>
-        <joint name="torso_to_${side}_upper_arm">
-          <hardwareInterface>hardware_interface/PositionJointInterface</hardwareInterface>
-        </joint>
-        <actuator name="torso_to_${side}_upper_arm_motor">
-          <mechanicalReduction>1</mechanicalReduction>
-        </actuator>
-      </transmission>
-    </joint>
-    <link name="${side}_forearm">
-      <visual>
-        <geometry><box size="0.06 0.06 0.25"/></geometry>
-        <material name="white"/>
-      </visual>
-      <collision>
-        <geometry><box size="0.06 0.06 0.25"/></geometry>
-      </collision>
-      <inertial>
-        <mass value="0.5"/>
-        <inertia ixx="0.002" ixy="0" ixz="0" iyy="0.002" iyz="0" izz="0.001"/>
-      </inertial>
-    </link>
-    <gazebo reference="${side}_forearm">
-      <material>white</material>
-      <mu1>0.9</mu1>
-      <mu2>0.9</mu2>
-    </gazebo>
-    <joint name="${side}_elbow" type="revolute">
-      <parent link="${side}_upper_arm"/>
-      <child link="${side}_forearm"/>
-      <origin xyz="0 0 -0.15"/>
-      <axis xyz="0 1 0"/>
-      <limit lower="-1.57" upper="1.57" effort="10.0" velocity="1.0"/>
-      <transmission name="${side}_elbow_trans">
-        <type>transmission_interface/SimpleTransmission</type>
-        <joint name="${side}_elbow">
-          <hardwareInterface>hardware_interface/PositionJointInterface</hardwareInterface>
-        </joint>
-        <actuator name="${side}_elbow_motor">
-          <mechanicalReduction>1</mechanicalReduction>
-        </actuator>
-      </transmission>
-    </joint>
-    <!-- Gripper base -->
-    <link name="${side}_gripper_base">
-      <visual>
-        <geometry><box size="0.08 0.08 0.04"/></geometry>
-        <material name="grey"/>
-      </visual>
-      <collision>
-        <geometry><box size="0.08 0.08 0.04"/></geometry>
-      </collision>
-      <inertial>
-        <mass value="0.2"/>
-        <inertia ixx="0.0002" ixy="0" ixz="0" iyy="0.0002" iyz="0" izz="0.0001"/>
-      </inertial>
-    </link>
-    <gazebo reference="${side}_gripper_base">
-      <material>grey</material>
-      <mu1>0.9</mu1>
-      <mu2>0.9</mu2>
-    </gazebo>
-    <joint name="${side}_wrist" type="revolute">
-      <parent link="${side}_forearm"/>
-      <child link="${side}_gripper_base"/>
-      <origin xyz="0 0 -0.125"/>
-      <axis xyz="1 0 0"/>
-      <limit lower="-1.57" upper="1.57" effort="10.0" velocity="1.0"/>
-      <transmission name="${side}_wrist_trans">
-        <type>transmission_interface/SimpleTransmission</type>
-        <joint name="${side}_wrist">
-          <hardwareInterface>hardware_interface/PositionJointInterface</hardwareInterface>
-        </joint>
-        <actuator name="${side}_wrist_motor">
-          <mechanicalReduction>1</mechanicalReduction>
-        </actuator>
-      </transmission>
-    </joint>
-    <!-- Gripper fingers -->
-    <link name="${side}_gripper_finger1">
-      <visual>
-        <geometry><box size="0.02 0.04 0.06"/></geometry>
-        <material name="black"/>
-      </visual>
-      <collision>
-        <geometry><box size="0.02 0.04 0.06"/></geometry>
-      </collision>
-      <inertial>
-        <mass value="0.05"/>
-        <inertia ixx="0.00005" ixy="0" ixz="0" iyy="0.00005" iyz="0" izz="0.00003"/>
-      </inertial>
-    </link>
-    <gazebo reference="${side}_gripper_finger1">
-      <material>black</material>
-      <mu1>0.9</mu1>
-      <mu2>0.9</mu2>
-    </gazebo>
-    <joint name="${side}_gripper_finger1_joint" type="prismatic">
-      <parent link="${side}_gripper_base"/>
-      <child link="${side}_gripper_finger1"/>
-      <origin xyz="0.03 0 -0.03"/>
-      <axis xyz="1 0 0"/>
-      <limit lower="-0.02" upper="0.02" effort="10.0" velocity="0.1"/>
-      <transmission name="${side}_gripper_finger1_trans">
-        <type>transmission_interface/SimpleTransmission</type>
-        <joint name="${side}_gripper_finger1_joint">
-          <hardwareInterface>hardware_interface/PositionJointInterface</hardwareInterface>
-        </joint>
-        <actuator name="${side}_gripper_finger1_motor">
-          <mechanicalReduction>1</mechanicalReduction>
-        </actuator>
-      </transmission>
-    </joint>
-    <link name="${side}_gripper_finger2">
-      <visual>
-        <geometry><box size="0.02 0.04 0.06"/></geometry>
-        <material name="black"/>
-      </visual>
-      <collision>
-        <geometry><box size="0.02 0.04 0.06"/></geometry>
-      </collision>
-      <inertial>
-        <mass value="0.05"/>
-        <inertia ixx="0.00005" ixy="0" ixz="0" iyy="0.00005" iyz="0" izz="0.00003"/>
-      </inertial>
-    </link>
-    <gazebo reference="${side}_gripper_finger2">
-      <material>black</material>
-      <mu1>0.9</mu1>
-      <mu2>0.9</mu2>
-    </gazebo>
-    <joint name="${side}_gripper_finger2_joint" type="prismatic">
-      <parent link="${side}_gripper_base"/>
-      <child link="${side}_gripper_finger2"/>
-      <origin xyz="-0.03 0 -0.03"/>
-      <axis xyz="1 0 0"/>
-      <limit lower="-0.02" upper="0.02" effort="10.0" velocity="0.1"/>
-      <transmission name="${side}_gripper_finger2_trans">
-        <type>transmission_interface/SimpleTransmission</type>
-        <joint name="${side}_gripper_finger2_joint">
-          <hardwareInterface>hardware_interface/PositionJointInterface</hardwareInterface>
-        </joint>
-        <actuator name="${side}_gripper_finger2_motor">
-          <mechanicalReduction>1</mechanicalReduction>
-        </actuator>
-      </transmission>
-    </joint>
-  </xacro:macro>
-  <!-- Macro for leg structure -->
-  <xacro:macro name="leg" params="side">
-    <link name="${side}_upper_leg">
-      <visual>
-        <geometry><box size="0.08 0.08 0.35"/></geometry>
-        <material name="black"/>
-      </visual>
-      <collision>
-        <geometry><box size="0.08 0.08 0.35"/></geometry>
-      </collision>
-      <inertial>
-        <mass value="1.5"/>
-        <inertia ixx="0.01" ixy="0" ixz="0" iyy="0.01" iyz="0" izz="0.005"/>
-      </inertial>
-    </link>
-    <gazebo reference="${side}_upper_leg">
-      <material>black</material>
-      <mu1>0.9</mu1>
-      <mu2>0.9</mu2>
-    </gazebo>
-    <xacro:property name="leg_offset_x" value="${side == 'left' ? 0.1 : -0.1}" />
-    <joint name="base_to_${side}_upper_leg" type="revolute">
-      <parent link="base_link"/>
-      <child link="${side}_upper_leg"/>
-      <origin xyz="${leg_offset_x} 0 0"/>
-      <axis xyz="1 0 0"/>
-      <limit lower="-1.57" upper="1.57" effort="10.0" velocity="1.0"/>
-      <transmission name="base_to_${side}_upper_leg_trans">
-        <type>transmission_interface/SimpleTransmission</type>
-        <joint name="base_to_${side}_upper_leg">
-          <hardwareInterface>hardware_interface/PositionJointInterface</hardwareInterface>
-        </joint>
-        <actuator name="base_to_${side}_upper_leg_motor">
-          <mechanicalReduction>1</mechanicalReduction>
-        </actuator>
-      </transmission>
-    </joint>
-    <link name="${side}_lower_leg">
-      <visual>
-        <geometry><box size="0.07 0.07 0.3"/></geometry>
-        <material name="grey"/>
-      </visual>
-      <collision>
-        <geometry><box size="0.07 0.07 0.3"/></geometry>
-      </collision>
-      <inertial>
-        <mass value="1.0"/>
-        <inertia ixx="0.005" ixy="0" ixz="0" iyy="0.005" iyz="0" izz="0.002"/>
-      </inertial>
-    </link>
-    <gazebo reference="${side}_lower_leg">
-      <material>grey</material>
-      <mu1>0.9</mu1>
-      <mu2>0.9</mu2>
-    </gazebo>
-    <joint name="${side}_knee" type="revolute">
-      <parent link="${side}_upper_leg"/>
-      <child link="${side}_lower_leg"/>
-      <origin xyz="0 0 -0.175"/>
-      <axis xyz="1 0 0"/>
-      <limit lower="0" upper="1.57" effort="10.0" velocity="1.0"/>
-      <transmission name="${side}_knee_trans">
-        <type>transmission_interface/SimpleTransmission</type>
-        <joint name="${side}_knee">
-          <hardwareInterface>hardware_interface/PositionJointInterface</hardwareInterface>
-        </joint>
-        <actuator name="${side}_knee_motor">
-          <mechanicalReduction>1</mechanicalReduction>
-        </actuator>
-      </transmission>
-    </joint>
-    <link name="${side}_foot">
-      <visual>
-        <geometry><box size="0.15 0.1 0.05"/></geometry>
-        <material name="grey"/>
-      </visual>
-      <collision>
-        <geometry><box size="0.15 0.1 0.05"/></geometry>
-      </collision>
-      <inertial>
-        <mass value="0.3"/>
-        <inertia ixx="0.0003" ixy="0" ixz="0" iyy="0.0003" iyz="0" izz="0.0001"/>
-      </inertial>
-    </link>
-    <gazebo reference="${side}_foot">
-      <material>grey</material>
-      <mu1>0.9</mu1>
-      <mu2>0.9</mu2>
-    </gazebo>
-    <joint name="${side}_ankle" type="revolute">
-      <parent link="${side}_lower_leg"/>
-      <child link="${side}_foot"/>
-      <origin xyz="0 0 -0.15"/>
-      <axis xyz="1 0 0"/>
-      <limit lower="-0.5" upper="0.5" effort="10.0" velocity="1.0"/>
-      <transmission name="${side}_ankle_trans">
-        <type>transmission_interface/SimpleTransmission</type>
-        <joint name="${side}_ankle">
-          <hardwareInterface>hardware_interface/PositionJointInterface</hardwareInterface>
-        </joint>
-        <actuator name="${side}_ankle_motor">
-          <mechanicalReduction>1</mechanicalReduction>
-        </actuator>
-      </transmission>
-    </joint>
-  </xacro:macro>
-  <!-- Base Link -->
-  <link name="base_link">
-    <visual>
-      <geometry><cylinder radius="0.15" length="0.1"/></geometry>
-      <material name="grey"/>
-    </visual>
-    <collision>
-      <geometry><cylinder radius="0.15" length="0.1"/></geometry>
-    </collision>
-    <inertial>
-      <mass value="5.0"/>
-      <inertia ixx="0.1" ixy="0" ixz="0" iyy="0.1" iyz="0" izz="0.05"/>
-    </inertial>
-  </link>
-  <gazebo reference="base_link">
-    <material>grey</material>
-    <mu1>0.9</mu1>
-    <mu2>0.9</mu2>
-    <inertial>
-      <mass>5.0</mass>
-      <inertia>
-        <ixx>0.1</ixx>
-        <ixy>0</ixy>
-        <ixz>0</ixz>
-        <iyy>0.1</iyy>
-        <iyz>0</iyz>
-        <izz>0.05</izz>
-      </inertia>
-    </inertial>
-  </gazebo>
-  <!-- Torso -->
-  <link name="torso">
-    <visual>
-      <geometry><box size="0.3 0.25 0.4"/></geometry>
-      <material name="black"/>
-    </visual>
-    <collision>
-      <geometry><box size="0.3 0.25 0.4"/></geometry>
-    </collision>
-    <inertial>
-      <mass value="3.0"/>
-      <inertia ixx="0.05" ixy="0" ixz="0" iyy="0.05" iyz="0" izz="0.03"/>
-    </inertial>
-  </link>
-  <gazebo reference="torso">
-    <material>black</material>
-    <mu1>0.9</mu1>
-    <mu2>0.9</mu2>
-    <inertial>
-      <mass>3.0</mass>
-      <inertia>
-        <ixx>0.05</ixx>
-        <ixy>0</ixy>
-        <ixz>0</ixz>
-        <iyy>0.05</iyy>
-        <iyz>0</iyz>
-        <izz>0.03</izz>
-      </inertia>
-    </inertial>
-  </gazebo>
-  <joint name="base_to_torso" type="fixed">
-    <parent link="base_link"/>
-    <child link="torso"/>
-    <origin xyz="0 0 0.25"/>
-  </joint>
-  <!-- Head -->
-  <link name="head">
-    <visual>
-      <geometry><box size="0.2 0.15 0.15"/></geometry>
-      <material name="white"/>
-    </visual>
-    <collision>
-      <geometry><box size="0.2 0.15 0.15"/></geometry>
-    </collision>
-    <inertial>
-      <mass value="1.0"/>
-      <inertia ixx="0.01" ixy="0" ixz="0" iyy="0.01" iyz="0" izz="0.01"/>
-    </inertial>
-  </link>
-  <gazebo reference="head">
-    <material>white</material>
-    <mu1>0.9</mu1>
-    <mu2>0.9</mu2>
-    <inertial>
-      <mass>1.0</mass>
-      <inertia>
-        <ixx>0.01</ixx>
-        <ixy>0</ixy>
-        <ixz>0</ixz>
-        <iyy>0.01</iyy>
-        <iyz>0</iyz>
-        <izz>0.01</izz>
-      </inertia>
-    </inertial>
-  </gazebo>
-  <joint name="torso_to_head" type="revolute">
-    <parent link="torso"/>
-    <child link="head"/>
-    <origin xyz="0 0 0.275"/>
-    <axis xyz="0 1 0"/>
-    <limit lower="-1.57" upper="1.57" effort="10.0" velocity="1.0"/>
-    <transmission name="torso_to_head_trans">
-      <type>transmission_interface/SimpleTransmission</type>
-      <joint name="torso_to_head">
-        <hardwareInterface>hardware_interface/PositionJointInterface</hardwareInterface>
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