Commit message: Attempt 2 at CORI Launch!

File: cori_ws/install/cori_description/share/cori_description/urdf/cori.urdf.xacro (robot description, xacro)
@@ -1 +1,534 @@
-/home/juptegraph/Workspaces/Robotics/Projects/CORI/cori_ws/src/cori_description/urdf/cori.urdf.xacro
+<?xml version="1.0"?>
+<robot name="cori" xmlns:xacro="http://www.ros.org/wiki/xacro">
+<!-- Materials -->
+<material name="body_material">
+  <color rgba="0.82 0.81 0.78 1.0"/> <!-- Light gray for body -->
+</material>
+<material name="joint_material">
+  <color rgba="0.35 0.35 0.35 1.0"/> <!-- Dark gray for joints -->
+</material>
+<material name="screen_material">
+  <color rgba="0.05 0.05 0.05 1.0"/> <!-- Black for screen -->
+</material>
+<material name="eye_material">
+  <color rgba="1.0 1.0 1.0 1.0"/> <!-- White for eyes -->
+</material>
+<!-- Joint Properties Macro -->
+<xacro:macro name="joint_properties">
+  <limit lower="-2.09" upper="2.09" effort="100.0" velocity="1.0"/>
+  <dynamics damping="0.7" friction="0.9"/>
+</xacro:macro>
+<!-- Base Link -->
+<link name="base_link">
+  <visual>
+    <geometry>
+      <cylinder radius="0.05" length="0.02"/>
+    </geometry>
+    <material name="joint_material"/>
+  </visual>
+  <collision>
+    <geometry>
+      <cylinder radius="0.05" length="0.02"/>
+    </geometry>
+  </collision>
+  <inertial>
+    <mass value="0.1"/>
+    <inertia ixx="0.001" ixy="0.0" ixz="0.0" iyy="0.001" iyz="0.0" izz="0.001"/>
+  </inertial>
+</link>
+<!-- Full Body Collision Link using STL -->
+<link name="full_body_collision">
+  <collision>
+    <geometry>
+<mesh filename="/home/juptegraph/Workspaces/Robotics/Projects/CORI/cori_ws/install/cori_description/share/cori_description/meshes/CORI_Solid.stl" scale="0.001 0.001 0.001"/>  </collision>
+</link>
+<joint name="body_collision_joint" type="fixed">
+  <parent link="base_link"/>
+  <child link="full_body_collision"/>
+  <origin xyz="0 0 0" rpy="0 0 0"/>
+</joint>
+<!-- Head Assembly -->
+<link name="head">
+  <visual>
+    <geometry>
+      <box size="0.28 0.2 0.14"/>
+    </geometry>
+    <material name="body_material"/>
+  </visual>
+  <!-- Removed individual collision - using full body STL instead -->
+  <inertial>
+    <mass value="1.5"/>
+    <inertia ixx="0.015" ixy="0.0" ixz="0.0" iyy="0.015" iyz="0.0" izz="0.015"/>
+  </inertial>
+</link>
+<joint name="neck_joint" type="revolute">
+  <parent link="base_link"/>
+  <child link="head"/>
+  <axis xyz="0 0 1"/>
+  <xacro:joint_properties/>
+  <origin xyz="0 0 0.38" rpy="0 0 0"/>
+</joint>
+<link name="screen">
+  <visual>
+    <geometry>
+      <box size="0.22 0.01 0.12"/>
+    </geometry>
+    <material name="screen_material"/>
+  </visual>
+  <inertial>
+    <mass value="0.1"/>
+    <inertia ixx="0.001" ixy="0.0" ixz="0.0" iyy="0.001" iyz="0.0" izz="0.001"/>
+  </inertial>
+</link>
+<joint name="screen_joint" type="fixed">
+  <parent link="head"/>
+  <child link="screen"/>
+  <origin xyz="0 0.1 0.02" rpy="0 0 0"/>
+</joint>
+<link name="left_eye">
+  <visual>
+    <geometry>
+      <sphere radius="0.015"/>
+    </geometry>
+    <material name="eye_material"/>
+  </visual>
+  <inertial>
+    <mass value="0.01"/>
+    <inertia ixx="0.0001" ixy="0.0" ixz="0.0" iyy="0.0001" iyz="0.0" izz="0.0001"/>
+  </inertial>
+</link>
+<joint name="left_eye_joint" type="fixed">
+  <parent link="screen"/>
+  <child link="left_eye"/>
+  <origin xyz="-0.08 0.02 0.02" rpy="0 0 0"/>
+</joint>
+<link name="right_eye">
+  <visual>
+    <geometry>
+      <sphere radius="0.015"/>
+    </geometry>
+    <material name="eye_material"/>
+  </visual>
+  <inertial>
+    <mass value="0.01"/>
+    <inertia ixx="0.0001" ixy="0.0" ixz="0.0" iyy="0.0001" iyz="0.0" izz="0.0001"/>
+  </inertial>
+</link>
+<joint name="right_eye_joint" type="fixed">
+  <parent link="screen"/>
+  <child link="right_eye"/>
+  <origin xyz="0.08 0.02 0.02" rpy="0 0 0"/>
+</joint>
+<!-- Torso Assembly -->
+<link name="torso">
+  <visual>
+    <geometry>
+      <box size="0.32 0.22 0.38"/>
+    </geometry>
+    <material name="body_material"/>
+  </visual>
+  <!-- Removed individual collision - using full body STL instead -->
+  <inertial>
+    <mass value="8.0"/>
+    <inertia ixx="0.08" ixy="0.0" ixz="0.0" iyy="0.08" iyz="0.0" izz="0.08"/>
+  </inertial>
+</link>
+<joint name="waist_joint" type="revolute">
+  <parent link="base_link"/>
+  <child link="torso"/>
+  <axis xyz="0 0 1"/>
+  <xacro:joint_properties/>
+  <origin xyz="0 0 0" rpy="0 0 0"/>
+</joint>
+<!-- Finger Macro -->
+<xacro:macro name="finger" params="hand name offset">
+  <link name="${hand}_finger_${name}">
+    <visual>
+      <geometry>
+        <cylinder radius="0.006" length="0.06"/>
+      </geometry>
+      <material name="joint_material"/>
+    </visual>
+    <collision>
+      <geometry>
+        <cylinder radius="0.006" length="0.06"/>
+      </geometry>
+    </collision>
+    <inertial>
+      <mass value="0.1"/>
+      <inertia ixx="0.0001" ixy="0.0" ixz="0.0" iyy="0.0001" iyz="0.0" izz="0.0001"/>
+    </inertial>
+  </link>
+  <joint name="${hand}_finger_${name}_joint" type="revolute">
+    <parent link="${hand}_hand_palm"/>
+    <child link="${hand}_finger_${name}"/>
+    <axis xyz="0 0 1"/>
+    <limit lower="0.0" upper="1.57" effort="50.0" velocity="0.5"/>
+    <dynamics damping="0.5" friction="0.7"/>
+    <origin xyz="${offset} 0 -0.025" rpy="0 0 0"/>
+  </joint>
+</xacro:macro>
+<!-- Left Arm -->
+<link name="left_arm_upper">
+  <visual>
+    <geometry>
+      <cylinder radius="0.0275" length="0.28"/>
+    </geometry>
+    <material name="body_material"/>
+  </visual>
+  <!-- Removed individual collision - using full body STL instead -->
+  <inertial>
+    <mass value="1.2"/>
+    <inertia ixx="0.012" ixy="0.0" ixz="0.0" iyy="0.012" iyz="0.0" izz="0.012"/>
+  </inertial>
+</link>
+<joint name="left_shoulder_joint" type="revolute">
+  <parent link="torso"/>
+  <child link="left_arm_upper"/>
+  <axis xyz="0 1 0"/>
+  <xacro:joint_properties/>
+  <origin xyz="-0.16 0 0.38" rpy="0 0 0"/>
+</joint>
+<link name="left_arm_elbow">
+  <visual>
+    <geometry>
+      <cylinder radius="0.0225" length="0.04"/>
+    </geometry>
+    <material name="joint_material"/>
+  </visual>
+  <collision>
+    <geometry>
+      <cylinder radius="0.0225" length="0.04"/>
+    </geometry>
+  </collision>
+  <inertial>
+    <mass value="0.3"/>
+    <inertia ixx="0.003" ixy="0.0" ixz="0.0" iyy="0.003" iyz="0.0" izz="0.003"/>
+  </inertial>
+</link>
+<joint name="left_elbow_joint" type="revolute">
+  <parent link="left_arm_upper"/>
+  <child link="left_arm_elbow"/>
+  <axis xyz="0 1 0"/>
+  <xacro:joint_properties/>
+  <origin xyz="0 0 0.14" rpy="0 0 0"/>
+</joint>
+<link name="left_arm_forearm">
+  <visual>
+    <geometry>
+      <cylinder radius="0.025" length="0.26"/>
+    </geometry>
+    <material name="body_material"/>
+  </visual>
+  <!-- Removed individual collision - using full body STL instead -->
+  <inertial>
+    <mass value="1.0"/>
+    <inertia ixx="0.01" ixy="0.0" ixz="0.0" iyy="0.01" iyz="0.0" izz="0.01"/>
+  </inertial>
+</link>
+<joint name="left_wrist_joint" type="revolute">
+  <parent link="left_arm_elbow"/>
+  <child link="left_arm_forearm"/>
+  <axis xyz="0 1 0"/>
+  <xacro:joint_properties/>
+  <origin xyz="0 0 0.02" rpy="0 0 0"/>
+</joint>
+<link name="left_hand_palm">
+  <visual>
+    <geometry>
+      <box size="0.085 0.06 0.025"/>
+    </geometry>
+    <material name="joint_material"/>
+  </visual>
+  <collision>
+    <geometry>
+      <box size="0.085 0.06 0.025"/>
+    </geometry>
+  </collision>
+  <inertial>
+    <mass value="0.6"/>
+    <inertia ixx="0.0015" ixy="0.0" ixz="0.0" iyy="0.0015" iyz="0.0" izz="0.0015"/>
+  </inertial>
+</link>
+<joint name="left_wrist_hand_joint" type="fixed">
+  <parent link="left_arm_forearm"/>
+  <child link="left_hand_palm"/>
+  <origin xyz="0 0 0.13" rpy="0 0 0"/>
+</joint>
+<!-- Left Hand Fingers -->
+<xacro:finger hand="left" name="1" offset="-0.02"/>
+<xacro:finger hand="left" name="2" offset="-0.0067"/>
+<xacro:finger hand="left" name="3" offset="0.0067"/>
+<xacro:finger hand="left" name="4" offset="0.02"/>
+<!-- Right Arm (Mirrored) -->
+<link name="right_arm_upper">
+  <visual>
+    <geometry>
+      <cylinder radius="0.0275" length="0.28"/>
+    </geometry>
+    <material name="body_material"/>
+  </visual>
+  <!-- Removed individual collision - using full body STL instead -->
+  <inertial>
+    <mass value="1.2"/>
+    <inertia ixx="0.012" ixy="0.0" ixz="0.0" iyy="0.012" iyz="0.0" izz="0.012"/>
+  </inertial>
+</link>
+<joint name="right_shoulder_joint" type="revolute">
+  <parent link="torso"/>
+  <child link="right_arm_upper"/>
+  <axis xyz="0 1 0"/>
+  <xacro:joint_properties/>
+  <origin xyz="0.16 0 0.38" rpy="0 0 0"/>
+</joint>
+<link name="right_arm_elbow">
+  <visual>
+    <geometry>
+      <cylinder radius="0.0225" length="0.04"/>
+    </geometry>
+    <material name="joint_material"/>
+  </visual>
+  <collision>
+    <geometry>
+      <cylinder radius="0.0225" length="0.04"/>
+    </geometry>
+  </collision>
+  <inertial>
+    <mass value="0.3"/>
+    <inertia ixx="0.003" ixy="0.0" ixz="0.0" iyy="0.003" iyz="0.0" izz="0.003"/>
+  </inertial>
+</link>
+<joint name="right_elbow_joint" type="revolute">
+  <parent link="right_arm_upper"/>
+  <child link="right_arm_elbow"/>
+  <axis xyz="0 1 0"/>
+  <xacro:joint_properties/>
+  <origin xyz="0 0 0.14" rpy="0 0 0"/>
+</joint>
+<link name="right_arm_forearm">
+  <visual>
+    <geometry>
+      <cylinder radius="0.025" length="0.26"/>
+    </geometry>
+    <material name="body_material"/>
+  </visual>
+  <!-- Removed individual collision - using full body STL instead -->
+  <inertial>
+    <mass value="1.0"/>
+    <inertia ixx="0.01" ixy="0.0" ixz="0.0" iyy="0.01" iyz="0.0" izz="0.01"/>
+  </inertial>
+</link>
+<joint name="right_wrist_joint" type="revolute">
+  <parent link="right_arm_elbow"/>
+  <child link="right_arm_forearm"/>
+  <axis xyz="0 1 0"/>
+  <xacro:joint_properties/>
+  <origin xyz="0 0 0.02" rpy="0 0 0"/>
+</joint>
+<link name="right_hand_palm">
+  <visual>
+    <geometry>
+      <box size="0.085 0.06 0.025"/>
+    </geometry>
+    <material name="joint_material"/>
+  </visual>
+  <collision>
+    <geometry>
+      <box size="0.085 0.06 0.025"/>
+    </geometry>
+  </collision>
+  <inertial>
+    <mass value="0.6"/>
+    <inertia ixx="0.0015" ixy="0.0" ixz="0.0" iyy="0.0015" iyz="0.0" izz="0.0015"/>
+  </inertial>
+</link>
+<joint name="right_wrist_hand_joint" type="fixed">
+  <parent link="right_arm_forearm"/>
+  <child link="right_hand_palm"/>
+  <origin xyz="0 0 0.13" rpy="0 0 0"/>
+</joint>
+<!-- Right Hand Fingers -->
+<xacro:finger hand="right" name="1" offset="-0.02"/>
+<xacro:finger hand="right" name="2" offset="-0.0067"/>
+<xacro:finger hand="right" name="3" offset="0.0067"/>
+<xacro:finger hand="right" name="4" offset="0.02"/>
+<!-- Left Leg -->
+<link name="left_leg_hip">
+  <visual>
+    <geometry>
+      <cylinder radius="0.03" length="0.04"/>
+    </geometry>
+    <material name="joint_material"/>
+  </visual>
+  <collision>
+    <geometry>
+      <cylinder radius="0.03" length="0.04"/>
+    </geometry>
+  </collision>
+  <inertial>
+    <mass value="1.0"/>
+    <inertia ixx="0.01" ixy="0.0" ixz="0.0" iyy="0.01" iyz="0.0" izz="0.01"/>
+  </inertial>
+</link>
+<joint name="left_hip_joint" type="revolute">
+  <parent link="torso"/>
+  <child link="left_leg_hip"/>
+  <axis xyz="0 1 0"/>
+  <xacro:joint_properties/>
+  <origin xyz="-0.08 0 -0.19" rpy="0 0 0"/>
+</joint>
+<link name="left_leg_thigh">
+  <visual>
+    <geometry>
+      <cylinder radius="0.03" length="0.35"/>
+    </geometry>
+    <material name="body_material"/>
+  </visual>
+  <!-- Removed individual collision - using full body STL instead -->
+  <inertial>
+    <mass value="1.5"/>
+    <inertia ixx="0.015" ixy="0.0" ixz="0.0" iyy="0.015" iyz="0.0" izz="0.015"/>
+  </inertial>
+</link>
+<joint name="left_knee_joint" type="revolute">
+  <parent link="left_leg_hip"/>
+  <child link="left_leg_thigh"/>
+  <axis xyz="0 1 0"/>
+  <xacro:joint_properties/>
+  <origin xyz="0 0 -0.175" rpy="0 0 0"/>
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
File: cori_ws/src/cori_description/urdf/cori.urdf.xacro (robot description, xacro)
@@ -41,7 +41,5 @@
   <collision>
     <geometry>
-      <mesh filename="meshes/CORI_Solid.stl" scale="0.001 0.001 0.001"/>
-    </geometry>
-  </collision>
+<mesh filename="/home/juptegraph/Workspaces/Robotics/Projects/CORI/cori_ws/install/cori_description/share/cori_description/meshes/CORI_Solid.stl" scale="0.001 0.001 0.001"/>  </collision>
 </link>
 <joint name="body_collision_joint" type="fixed">

Commit message: Successful CORI build, need to reduce STL size for rigidbody. Current, too large, need to be scaled down. Also, address Nvidia driver issues, missmatch between Gazebo Ignition and existing driver config.

File: cori_ws/install/cori_description/share/cori_description/urdf/cori.urdf.xacro (robot description, xacro)
@@ -41,5 +41,7 @@
   <collision>
     <geometry>
-<mesh filename="/home/juptegraph/Workspaces/Robotics/Projects/CORI/cori_ws/install/cori_description/share/cori_description/meshes/CORI_Solid.stl" scale="0.001 0.001 0.001"/>  </collision>
+      <!-- <mesh filename="/home/juptegraph/Workspaces/Robotics/Projects/CORI/cori_ws/src/cori_description/meshes/CORI_Solid.stl"/>     -->
+    </geometry>
+  </collision>
 </link>
 <joint name="body_collision_joint" type="fixed">
@@ -530,5 +532,5 @@
 <gazebo>
   <plugin name="ignition::gazebo::systems::JointStatePublisher" filename="ignition-gazebo-joint-state-publisher-system"/>
-  <plugin name="ignition::gazebo::systems::JointPositionController" filename="ignition-gazebo-joint-position-controller-system"/>
+  <!-- <plugin name="ignition::gazebo::systems::JointPositionController" filename="ignition-gazebo-joint-position-controller-system"/> -->
 </gazebo>
 </robot>

Commit message: Resolved driver issues, recorded CORI in Gazebo with objects + gravity. Backed up.

File: cori_ws/install/cori_description/share/cori_description/urdf/cori.urdf.xacro (robot description, xacro)
@@ -37,11 +37,15 @@
   </inertial>
 </link>
-<!-- Full Body Collision Link using STL -->
+<!-- Full Body Collision Link - FIXED -->
 <link name="full_body_collision">
   <collision>
     <geometry>
-      <!-- <mesh filename="/home/juptegraph/Workspaces/Robotics/Projects/CORI/cori_ws/src/cori_description/meshes/CORI_Solid.stl"/>     -->
-    </geometry>
-  </collision>
+      <box size="0.4 0.3 1.5"/>
+    </geometry>
+  </collision>
+  <inertial>
+    <mass value="5.0"/>
+    <inertia ixx="0.1" ixy="0.0" ixz="0.0" iyy="0.1" iyz="0.0" izz="0.1"/>
+  </inertial>
 </link>
 <joint name="body_collision_joint" type="fixed">

Commit message: Connected Color Detection Node to CORI. Outputing to live terminal feed. Created killall and build programs to enable user "run modes".

File: cori_ws/install/cori_description/share/cori_description/urdf/cori.urdf.xacro (robot description, xacro)
@@ -110,4 +110,53 @@
     </inertial>
   </link>
+  <!-- Camera Link -->
+<link name="camera_link">
+  <visual>
+    <geometry>
+      <box size="0.02 0.05 0.02"/>
+    </geometry>
+    <material name="joint_material"/>
+  </visual>
+  <collision>
+    <geometry>
+      <box size="0.02 0.05 0.02"/>
+    </geometry>
+  </collision>
+  <inertial>
+    <mass value="0.01"/>
+    <inertia ixx="0.0001" ixy="0.0" ixz="0.0" iyy="0.0001" iyz="0.0" izz="0.0001"/>
+  </inertial>
+</link>
+<joint name="head_to_camera" type="fixed">
+  <parent link="head"/>
+  <child link="camera_link"/>
+  <origin xyz="0.08 0 0.02" rpy="0 0 0"/>
+</joint>
+<!-- Camera Sensor
+<gazebo reference="camera_link">
+  <sensor type="camera" name="head_camera">
+    <update_rate>30.0</update_rate>
+    <camera name="head_camera">
+      <horizontal_fov>1.3962634</horizontal_fov>
+      <image>
+        <width>800</width>
+        <height>600</height>
+        <format>R8G8B8</format>
+      </image>
+      <clip>
+        <near>0.02</near>
+        <far>300</far>
+      </clip>
+    </camera>
+    <plugin name="camera_controller" filename="libgazebo_ros_camera.so">
+      <alwaysOn>true</alwaysOn>
+      <updateRate>0.0</updateRate>
+      <cameraName>cori/camera</cameraName>
+      <imageTopicName>image_raw</imageTopicName>
+      <cameraInfoTopicName>camera_info</cameraInfoTopicName>
+      <frameName>camera_link</frameName>
+    </plugin>
+  </sensor>
+</gazebo> -->
   <joint name="head_to_screen" type="fixed">
     <parent link="head"/>
