Commit message: Fully embodied CORI urdf is now rendered in Gazebo... seperate joints and all!

File: cori_ws/install/cori_description/share/cori_description/urdf/cori.urdf.xacro (robot description, xacro)
@@ -2,30 +2,51 @@
 <robot xmlns:xacro="http://www.ros.org/wiki/xacro" name="cori">
   <!-- Materials -->
-  <material name="body_material">
-    <color rgba="0.82 0.81 0.78 1.0"/> <!-- Light gray for body -->
+  <material name="cori_material">
+    <color rgba="0.7 0.7 0.7 1.0"/>
   </material>
-  <material name="joint_material">
-    <color rgba="0.35 0.35 0.35 1.0"/> <!-- Dark gray for joints -->
-  </material>
-  <material name="screen_material">
-    <color rgba="0.05 0.05 0.05 1.0"/> <!-- Black for screen -->
-  </material>
-  <material name="eye_material">
-    <color rgba="1.0 1.0 1.0 1.0"/> <!-- White for eyes -->
-  </material>
-  <material name="invisible">
-    <color rgba="0.0 0.0 0.0 0.0"/> <!-- Transparent -->
+  <material name="head_material">
+    <color rgba="0.3 0.3 0.3 1.0"/>
   </material>
   <!-- Base Link -->
   <link name="base_link">
-    <visual>
-      <geometry>
-        <cylinder radius="0.15" length="0.05"/>
-      </geometry>
-      <material name="invisible"/> <!-- Make base invisible -->
-    </visual>
-    <collision>
-      <geometry>
-        <cylinder radius="0.15" length="0.05"/>
+    <inertial>
+      <mass value="0.1"/>
+      <inertia ixx="0.001" ixy="0.0" ixz="0.0" iyy="0.001" iyz="0.0" izz="0.001"/>
+    </inertial>
+  </link>
+  <!-- Torso -->
+  <link name="torso">
+    <visual>
+      <geometry>
+        <mesh filename="file:///home/juptegraph/Workspaces/Robotics/Projects/CORI/cori_ws/src/cori_description/meshes/cori_body_v1.0/cori_torso.stl" scale="0.4 0.4 0.4"/>
+      </geometry>
+      <material name="cori_material"/>
+    </visual>
+    <collision>
+      <geometry>
+        <mesh filename="file:///home/juptegraph/Workspaces/Robotics/Projects/CORI/cori_ws/src/cori_description/meshes/cori_body_v1.0/cori_torso.stl" scale="0.4 0.4 0.4"/>
+      </geometry>
+    </collision>
+    <inertial>
+      <mass value="5.0"/>
+      <inertia ixx="0.1" ixy="0.0" ixz="0.0" iyy="0.1" iyz="0.0" izz="0.1"/>
+    </inertial>
+  </link>
+  <joint name="base_to_torso" type="fixed">
+    <parent link="base_link"/>
+    <child link="torso"/>
+    <origin xyz="0 0 0" rpy="0 0 0"/>
+  </joint>
+  <!-- HEAD - MOVEABLE! -->
+  <link name="head">
+    <visual>
+      <geometry>
+        <mesh filename="file:///home/juptegraph/Workspaces/Robotics/Projects/CORI/cori_ws/src/cori_description/meshes/cori_body_v1.0/cori_head.stl" scale="0.4 0.4 0.4"/>
+      </geometry>
+      <material name="head_material"/>
+    </visual>
+    <collision>
+      <geometry>
+        <mesh filename="file:///home/juptegraph/Workspaces/Robotics/Projects/CORI/cori_ws/src/cori_description/meshes/cori_body_v1.0/cori_head.stl" scale="0.4 0.4 0.4"/>
       </geometry>
     </collision>
@@ -35,54 +56,355 @@
     </inertial>
   </link>
-  <!-- Full Body Collision Link - THIS WILL SHOW YOUR STL MESH -->
-  <link name="full_body_collision">
-    <visual>
-      <geometry>
-        <mesh filename="file:///home/juptegraph/Workspaces/Robotics/Projects/CORI/cori_ws/src/cori_description/meshes/CORI_Solid.stl" scale="0.03 0.03 0.03"/>
-      </geometry>
-      <material name="body_material"/>
-    </visual>
-    <collision>
-      <geometry>
-        <mesh filename="file:///home/juptegraph/Workspaces/Robotics/Projects/CORI/cori_ws/src/cori_description/meshes/CORI_Solid.stl" scale="0.03 0.03 0.03"/>
-      </geometry>
-    </collision>
-    <inertial>
-      <mass value="50.0"/>
-      <inertia ixx="2.0" ixy="0.0" ixz="0.0" iyy="2.0" iyz="0.0" izz="1.0"/>
-    </inertial>
-  </link>
-  <!-- Joint connecting base to full body -->
-  <joint name="base_to_body" type="fixed">
-    <parent link="base_link"/>
-    <child link="full_body_collision"/>
-    <origin xyz="-0.07 0 0.025" rpy="0 0 1.57"/>
-  </joint>
-  <!-- Torso - Made invisible -->
-  <link name="torso">
-    <visual>
-      <geometry>
-        <cylinder radius="0.12" length="0.25"/>
-      </geometry>
-      <material name="invisible"/>
-    </visual>
-    <inertial>
-      <mass value="5.0"/>
-      <inertia ixx="0.05" ixy="0.0" ixz="0.0" iyy="0.05" iyz="0.0" izz="0.02"/>
-    </inertial>
-  </link>
-  <joint name="body_to_torso" type="fixed">
-    <parent link="full_body_collision"/>
-    <child link="torso"/>
-    <origin xyz="0 0 0.125" rpy="0 0 0"/>
-  </joint>
-  <!-- Head - Made invisible -->
-  <link name="head">
-    <visual>
-      <geometry>
-        <sphere radius="0.08"/>
-      </geometry>
-      <material name="invisible"/>
-    </visual>
+  <!-- HEAD JOINT - This makes the head turn! -->
+  <joint name="head_joint" type="revolute">
+    <parent link="torso"/>
+    <child link="head"/>
+    <origin xyz="0 0 0" rpy="0 0 0"/>
+    <axis xyz="0 0 1"/>
+    <limit lower="-3.14159" upper="3.14159" effort="5" velocity="1.0"/>
+    <dynamics damping="0.2" friction="0.1"/>
+  </joint>
+  <!-- Camera (virtual - attached to head) -->
+  <link name="camera_link">
+    <visual>
+      <geometry>
+        <box size="0.01 0.02 0.005"/>
+      </geometry>
+      <material name="head_material"/>
+    </visual>
+    <inertial>
+      <mass value="0.01"/>
+      <inertia ixx="0.0001" ixy="0.0" ixz="0.0" iyy="0.0001" iyz="0.0" izz="0.0001"/>
+    </inertial>
+  </link>
+  <joint name="head_to_camera" type="fixed">
+    <parent link="head"/>
+    <child link="camera_link"/>
+    <origin xyz="0.05 0 0.02" rpy="0 0 0"/>
+  </joint>
+  <!-- LEFT ARM ASSEMBLY -->
+  <link name="left_upper_arm">
+    <visual>
+      <geometry>
+        <mesh filename="file:///home/juptegraph/Workspaces/Robotics/Projects/CORI/cori_ws/src/cori_description/meshes/cori_body_v1.0/cori_left_upper_arm.stl" scale="0.4 0.4 0.4"/>
+      </geometry>
+      <material name="cori_material"/>
+    </visual>
+    <collision>
+      <geometry>
+        <mesh filename="file:///home/juptegraph/Workspaces/Robotics/Projects/CORI/cori_ws/src/cori_description/meshes/cori_body_v1.0/cori_left_upper_arm.stl" scale="0.4 0.4 0.4"/>
+      </geometry>
+    </collision>
+    <inertial>
+      <mass value="0.8"/>
+      <inertia ixx="0.01" ixy="0.0" ixz="0.0" iyy="0.01" iyz="0.0" izz="0.005"/>
+    </inertial>
+  </link>
+  <joint name="torso_to_left_upper_arm" type="fixed">
+    <parent link="torso"/>
+    <child link="left_upper_arm"/>
+    <origin xyz="0 0 0" rpy="0 0 0"/>
+  </joint>
+  <link name="left_forearm">
+    <visual>
+      <geometry>
+        <mesh filename="file:///home/juptegraph/Workspaces/Robotics/Projects/CORI/cori_ws/src/cori_description/meshes/cori_body_v1.0/cori_left_forearm.stl" scale="0.4 0.4 0.4"/>
+      </geometry>
+      <material name="cori_material"/>
+    </visual>
+    <collision>
+      <geometry>
+        <mesh filename="file:///home/juptegraph/Workspaces/Robotics/Projects/CORI/cori_ws/src/cori_description/meshes/cori_body_v1.0/cori_left_forearm.stl" scale="0.4 0.4 0.4"/>
+      </geometry>
+    </collision>
+    <inertial>
+      <mass value="0.6"/>
+      <inertia ixx="0.008" ixy="0.0" ixz="0.0" iyy="0.008" iyz="0.0" izz="0.004"/>
+    </inertial>
+  </link>
+  <joint name="left_upper_arm_to_forearm" type="fixed">
+    <parent link="left_upper_arm"/>
+    <child link="left_forearm"/>
+    <origin xyz="0 0 0" rpy="0 0 0"/>
+  </joint>
+  <link name="left_hand">
+    <visual>
+      <geometry>
+        <mesh filename="file:///home/juptegraph/Workspaces/Robotics/Projects/CORI/cori_ws/src/cori_description/meshes/cori_body_v1.0/cori_left_hand.stl" scale="0.4 0.4 0.4"/>
+      </geometry>
+      <material name="cori_material"/>
+    </visual>
+    <collision>
+      <geometry>
+        <mesh filename="file:///home/juptegraph/Workspaces/Robotics/Projects/CORI/cori_ws/src/cori_description/meshes/cori_body_v1.0/cori_left_hand.stl" scale="0.4 0.4 0.4"/>
+      </geometry>
+    </collision>
+    <inertial>
+      <mass value="0.3"/>
+      <inertia ixx="0.005" ixy="0.0" ixz="0.0" iyy="0.005" iyz="0.0" izz="0.005"/>
+    </inertial>
+  </link>
+  <joint name="left_forearm_to_hand" type="fixed">
+    <parent link="left_forearm"/>
+    <child link="left_hand"/>
+    <origin xyz="0 0 0" rpy="0 0 0"/>
+  </joint>
+  <!-- RIGHT ARM ASSEMBLY -->
+  <link name="right_upper_arm">
+    <visual>
+      <geometry>
+        <mesh filename="file:///home/juptegraph/Workspaces/Robotics/Projects/CORI/cori_ws/src/cori_description/meshes/cori_body_v1.0/cori_right_upper_arm.stl" scale="0.4 0.4 0.4"/>
+      </geometry>
+      <material name="cori_material"/>
+    </visual>
+    <collision>
+      <geometry>
+        <mesh filename="file:///home/juptegraph/Workspaces/Robotics/Projects/CORI/cori_ws/src/cori_description/meshes/cori_body_v1.0/cori_right_upper_arm.stl" scale="0.4 0.4 0.4"/>
+      </geometry>
+    </collision>
+    <inertial>
+      <mass value="0.8"/>
+      <inertia ixx="0.01" ixy="0.0" ixz="0.0" iyy="0.01" iyz="0.0" izz="0.005"/>
+    </inertial>
+  </link>
+  <joint name="torso_to_right_upper_arm" type="fixed">
+    <parent link="torso"/>
+    <child link="right_upper_arm"/>
+    <origin xyz="0 0 0" rpy="0 0 0"/>
+  </joint>
+  <link name="right_forearm">
+    <visual>
+      <geometry>
+        <mesh filename="file:///home/juptegraph/Workspaces/Robotics/Projects/CORI/cori_ws/src/cori_description/meshes/cori_body_v1.0/cori_right_forearm.stl" scale="0.4 0.4 0.4"/>
+      </geometry>
+      <material name="cori_material"/>
+    </visual>
+    <collision>
+      <geometry>
+        <mesh filename="file:///home/juptegraph/Workspaces/Robotics/Projects/CORI/cori_ws/src/cori_description/meshes/cori_body_v1.0/cori_right_forearm.stl" scale="0.4 0.4 0.4"/>
+      </geometry>
+    </collision>
+    <inertial>
+      <mass value="0.6"/>
+      <inertia ixx="0.008" ixy="0.0" ixz="0.0" iyy="0.008" iyz="0.0" izz="0.004"/>
+    </inertial>
+  </link>
+  <joint name="right_upper_arm_to_forearm" type="fixed">
+    <parent link="right_upper_arm"/>
+    <child link="right_forearm"/>
+    <origin xyz="0 0 0" rpy="0 0 0"/>
+  </joint>
+  <link name="right_hand">
+    <visual>
+      <geometry>
+        <mesh filename="file:///home/juptegraph/Workspaces/Robotics/Projects/CORI/cori_ws/src/cori_description/meshes/cori_body_v1.0/cori_right_hand.stl" scale="0.4 0.4 0.4"/>
+      </geometry>
+      <material name="cori_material"/>
+    </visual>
+    <collision>
+      <geometry>
+        <mesh filename="file:///home/juptegraph/Workspaces/Robotics/Projects/CORI/cori_ws/src/cori_description/meshes/cori_body_v1.0/cori_right_hand.stl" scale="0.4 0.4 0.4"/>
+      </geometry>
+    </collision>
+    <inertial>
+      <mass value="0.3"/>
+      <inertia ixx="0.005" ixy="0.0" ixz="0.0" iyy="0.005" iyz="0.0" izz="0.005"/>
+    </inertial>
+  </link>
+  <joint name="right_forearm_to_hand" type="fixed">
+    <parent link="right_forearm"/>
+    <child link="right_hand"/>
+    <origin xyz="0 0 0" rpy="0 0 0"/>
+  </joint>
+  <!-- LEFT LEG ASSEMBLY -->
+  <link name="left_thigh">
+    <visual>
+      <geometry>
+        <mesh filename="file:///home/juptegraph/Workspaces/Robotics/Projects/CORI/cori_ws/src/cori_description/meshes/cori_body_v1.0/cori_left_thigh.stl" scale="0.4 0.4 0.4"/>
+      </geometry>
+      <material name="cori_material"/>
+    </visual>
+    <collision>
+      <geometry>
+        <mesh filename="file:///home/juptegraph/Workspaces/Robotics/Projects/CORI/cori_ws/src/cori_description/meshes/cori_body_v1.0/cori_left_thigh.stl" scale="0.4 0.4 0.4"/>
+      </geometry>
+    </collision>
+    <inertial>
+      <mass value="1.2"/>
+      <inertia ixx="0.02" ixy="0.0" ixz="0.0" iyy="0.02" iyz="0.0" izz="0.01"/>
+    </inertial>
+  </link>
+  <joint name="torso_to_left_thigh" type="fixed">
+    <parent link="torso"/>
+    <child link="left_thigh"/>
+    <origin xyz="0 0 0" rpy="0 0 0"/>
+  </joint>
+  <link name="left_shin">
+    <visual>
+      <geometry>
+        <mesh filename="file:///home/juptegraph/Workspaces/Robotics/Projects/CORI/cori_ws/src/cori_description/meshes/cori_body_v1.0/cori_left_shin.stl" scale="0.4 0.4 0.4"/>
+      </geometry>
+      <material name="cori_material"/>
+    </visual>
+    <collision>
+      <geometry>
+        <mesh filename="file:///home/juptegraph/Workspaces/Robotics/Projects/CORI/cori_ws/src/cori_description/meshes/cori_body_v1.0/cori_left_shin.stl" scale="0.4 0.4 0.4"/>
+      </geometry>
+    </collision>
+    <inertial>
+      <mass value="0.8"/>
+      <inertia ixx="0.01" ixy="0.0" ixz="0.0" iyy="0.01" iyz="0.0" izz="0.005"/>
+    </inertial>
+  </link>
+  <joint name="left_thigh_to_shin" type="fixed">
+    <parent link="left_thigh"/>
+    <child link="left_shin"/>
+    <origin xyz="0 0 0" rpy="0 0 0"/>
+  </joint>
+  <link name="left_knee">
+    <visual>
+      <geometry>
+        <mesh filename="file:///home/juptegraph/Workspaces/Robotics/Projects/CORI/cori_ws/src/cori_description/meshes/cori_body_v1.0/cori_left_knee.stl" scale="0.4 0.4 0.4"/>
+      </geometry>
+      <material name="cori_material"/>
+    </visual>
+    <collision>
+      <geometry>
+        <mesh filename="file:///home/juptegraph/Workspaces/Robotics/Projects/CORI/cori_ws/src/cori_description/meshes/cori_body_v1.0/cori_left_knee.stl" scale="0.4 0.4 0.4"/>
+      </geometry>
+    </collision>
+    <inertial>
+      <mass value="0.3"/>
+      <inertia ixx="0.005" ixy="0.0" ixz="0.0" iyy="0.005" iyz="0.0" izz="0.005"/>
+    </inertial>
+  </link>
+  <joint name="left_shin_to_knee" type="fixed">
+    <parent link="left_shin"/>
+    <child link="left_knee"/>
+    <origin xyz="0 0 0" rpy="0 0 0"/>
+  </joint>
+  <link name="left_foot">
+    <visual>
+      <geometry>
+        <mesh filename="file:///home/juptegraph/Workspaces/Robotics/Projects/CORI/cori_ws/src/cori_description/meshes/cori_body_v1.0/cori_left_foot.stl" scale="0.4 0.4 0.4"/>
+      </geometry>
+      <material name="cori_material"/>
+    </visual>
+    <collision>
+      <geometry>
+        <mesh filename="file:///home/juptegraph/Workspaces/Robotics/Projects/CORI/cori_ws/src/cori_description/meshes/cori_body_v1.0/cori_left_foot.stl" scale="0.4 0.4 0.4"/>
+      </geometry>
+    </collision>
+    <inertial>
+      <mass value="0.5"/>
+      <inertia ixx="0.005" ixy="0.0" ixz="0.0" iyy="0.005" iyz="0.0" izz="0.005"/>
+    </inertial>
+  </link>
+  <joint name="left_knee_to_foot" type="fixed">
+    <parent link="left_knee"/>
+    <child link="left_foot"/>
+    <origin xyz="0 0 0" rpy="0 0 0"/>
+  </joint>
+  <!-- RIGHT LEG ASSEMBLY -->
+  <link name="right_thigh">
+    <visual>
+      <geometry>
+        <mesh filename="file:///home/juptegraph/Workspaces/Robotics/Projects/CORI/cori_ws/src/cori_description/meshes/cori_body_v1.0/cori_right_thigh.stl" scale="0.4 0.4 0.4"/>
+      </geometry>
+      <material name="cori_material"/>
+    </visual>
+    <collision>
+      <geometry>
+        <mesh filename="file:///home/juptegraph/Workspaces/Robotics/Projects/CORI/cori_ws/src/cori_description/meshes/cori_body_v1.0/cori_right_thigh.stl" scale="0.4 0.4 0.4"/>
+      </geometry>
+    </collision>
+    <inertial>
+      <mass value="1.2"/>
+      <inertia ixx="0.02" ixy="0.0" ixz="0.0" iyy="0.02" iyz="0.0" izz="0.01"/>
+    </inertial>
+  </link>
+  <joint name="torso_to_right_thigh" type="fixed">
+    <parent link="torso"/>
+    <child link="right_thigh"/>
+    <origin xyz="0 0 0" rpy="0 0 0"/>
+  </joint>
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