Commit message: Fully articulating head with URDF... might need to adjust head origin for adaptive turning

File: cori_ws/src/cori_description/urdf/cori.urdf.xacro (robot description, xacro)
@@ -1,34 +1,39 @@
 <?xml version="1.0"?>
 <robot xmlns:xacro="http://www.ros.org/wiki/xacro" name="cori">
-  <!-- Materials -->
-  <material name="cori_material">
-    <color rgba="0.7 0.7 0.7 1.0"/>
+  <material name="cori_white">
+    <color rgba="0.95 0.95 0.95 1.0"/>
   </material>
-  <material name="head_material">
-    <color rgba="0.3 0.3 0.3 1.0"/>
+  <material name="cori_head">
+    <color rgba="0.85 0.85 1.0 1.0"/>
   </material>
-  <!-- Base Link -->
   <link name="base_link">
     <inertial>
-      <mass value="0.1"/>
-      <inertia ixx="0.001" ixy="0.0" ixz="0.0" iyy="0.001" iyz="0.0" izz="0.001"/>
-    </inertial>
-  </link>
-  <!-- Torso -->
+      <mass value="30.0"/>
+      <origin xyz="0 0 0"/>
+      <inertia ixx="2.0" ixy="0.0" ixz="0.0" iyy="2.0" iyz="0.0" izz="2.0"/>
+    </inertial>
+    <collision>
+      <geometry>
+        <box size="0.4 0.4 0.05"/>
+      </geometry>
+    </collision>
+  </link>
   <link name="torso">
     <visual>
-      <geometry>
-        <mesh filename="file:///home/juptegraph/Workspaces/Robotics/Projects/CORI/cori_ws/src/cori_description/meshes/cori_body_v1.0/cori_torso.stl" scale="0.4 0.4 0.4"/>
-      </geometry>
-      <material name="cori_material"/>
-    </visual>
-    <collision>
-      <geometry>
-        <mesh filename="file:///home/juptegraph/Workspaces/Robotics/Projects/CORI/cori_ws/src/cori_description/meshes/cori_body_v1.0/cori_torso.stl" scale="0.4 0.4 0.4"/>
-      </geometry>
-    </collision>
-    <inertial>
-      <mass value="5.0"/>
-      <inertia ixx="0.1" ixy="0.0" ixz="0.0" iyy="0.1" iyz="0.0" izz="0.1"/>
+      <origin xyz="0 0 0" rpy="0 0 0"/>
+      <geometry>
+        <mesh filename="file:///home/juptegraph/Workspaces/Robotics/Projects/CORI/cori_ws/src/cori_description/meshes/cori_body_v1.0/cori_torso.stl" scale="0.35 0.35 0.35"/>
+      </geometry>
+      <material name="cori_white"/>
+    </visual>
+    <collision>
+      <geometry>
+        <box size="0.2 0.12 0.3"/>
+      </geometry>
+    </collision>
+    <inertial>
+      <mass value="12.0"/>
+      <origin xyz="0 0 0"/>
+      <inertia ixx="0.4" ixy="0.0" ixz="0.0" iyy="0.4" iyz="0.0" izz="0.25"/>
     </inertial>
   </link>
@@ -36,67 +41,74 @@
     <parent link="base_link"/>
     <child link="torso"/>
-    <origin xyz="0 0 0" rpy="0 0 0"/>
-  </joint>
-  <!-- HEAD - MOVEABLE! -->
+    <origin xyz="0 0 0.15" rpy="0 0 0"/>
+  </joint>
   <link name="head">
     <visual>
-      <geometry>
-        <mesh filename="file:///home/juptegraph/Workspaces/Robotics/Projects/CORI/cori_ws/src/cori_description/meshes/cori_body_v1.0/cori_head.stl" scale="0.4 0.4 0.4"/>
-      </geometry>
-      <material name="head_material"/>
-    </visual>
-    <collision>
-      <geometry>
-        <mesh filename="file:///home/juptegraph/Workspaces/Robotics/Projects/CORI/cori_ws/src/cori_description/meshes/cori_body_v1.0/cori_head.stl" scale="0.4 0.4 0.4"/>
-      </geometry>
-    </collision>
-    <inertial>
-      <mass value="1.0"/>
-      <inertia ixx="0.01" ixy="0.0" ixz="0.0" iyy="0.01" iyz="0.0" izz="0.01"/>
-    </inertial>
-  </link>
-  <!-- HEAD JOINT - This makes the head turn! -->
+      <origin xyz="0 0 0" rpy="0 0 0"/>
+      <geometry>
+        <mesh filename="file:///home/juptegraph/Workspaces/Robotics/Projects/CORI/cori_ws/src/cori_description/meshes/cori_body_v1.0/cori_head.stl" scale="0.35 0.35 0.35"/>
+      </geometry>
+      <material name="cori_head"/>
+    </visual>
+    <collision>
+      <geometry>
+        <box size="0.12 0.12 0.12"/>
+      </geometry>
+    </collision>
+    <inertial>
+      <mass value="1.8"/>
+      <origin xyz="0 0 0"/>
+      <inertia ixx="0.018" ixy="0.0" ixz="0.0" iyy="0.018" iyz="0.0" izz="0.018"/>
+    </inertial>
+  </link>
   <joint name="head_joint" type="revolute">
     <parent link="torso"/>
     <child link="head"/>
-    <origin xyz="0 0 0" rpy="0 0 0"/>
+    <origin xyz="0 0 0" rpy="0 0 0"/>  <!-- Zero distance -->
     <axis xyz="0 0 1"/>
-    <limit lower="-3.14159" upper="3.14159" effort="5" velocity="1.0"/>
-    <dynamics damping="0.2" friction="0.1"/>
-  </joint>
-  <!-- Camera (virtual - attached to head) -->
-  <link name="camera_link">
-    <visual>
-      <geometry>
-        <box size="0.01 0.02 0.005"/>
-      </geometry>
-      <material name="head_material"/>
-    </visual>
-    <inertial>
-      <mass value="0.01"/>
-      <inertia ixx="0.0001" ixy="0.0" ixz="0.0" iyy="0.0001" iyz="0.0" izz="0.0001"/>
-    </inertial>
-  </link>
-  <joint name="head_to_camera" type="fixed">
-    <parent link="head"/>
-    <child link="camera_link"/>
-    <origin xyz="0.05 0 0.02" rpy="0 0 0"/>
-  </joint>
-  <!-- LEFT ARM ASSEMBLY -->
+    <limit lower="-1.8" upper="1.8" effort="80" velocity="2.5"/>
+    <dynamics damping="1.8" friction="0.9"/>
+  </joint>
+  <link name="pelvis">
+    <visual>
+      <origin xyz="0 0 0" rpy="0 0 0"/>
+      <geometry>
+        <mesh filename="file:///home/juptegraph/Workspaces/Robotics/Projects/CORI/cori_ws/src/cori_description/meshes/cori_body_v1.0/cori_pelvis.stl" scale="0.35 0.35 0.35"/>
+      </geometry>
+      <material name="cori_white"/>
+    </visual>
+    <collision>
+      <geometry>
+        <box size="0.18 0.22 0.08"/>
+      </geometry>
+    </collision>
+    <inertial>
+      <mass value="2.5"/>
+      <origin xyz="0 0 0"/>
+      <inertia ixx="0.025" ixy="0.0" ixz="0.0" iyy="0.03" iyz="0.0" izz="0.025"/>
+    </inertial>
+  </link>
+  <joint name="torso_to_pelvis" type="fixed">
+    <parent link="torso"/>
+    <child link="pelvis"/>
+    <origin xyz="0 0 0" rpy="0 0 0"/>  <!-- Zero distance -->
+  </joint>
   <link name="left_upper_arm">
     <visual>
-      <geometry>
-        <mesh filename="file:///home/juptegraph/Workspaces/Robotics/Projects/CORI/cori_ws/src/cori_description/meshes/cori_body_v1.0/cori_left_upper_arm.stl" scale="0.4 0.4 0.4"/>
-      </geometry>
-      <material name="cori_material"/>
-    </visual>
-    <collision>
-      <geometry>
-        <mesh filename="file:///home/juptegraph/Workspaces/Robotics/Projects/CORI/cori_ws/src/cori_description/meshes/cori_body_v1.0/cori_left_upper_arm.stl" scale="0.4 0.4 0.4"/>
-      </geometry>
-    </collision>
-    <inertial>
-      <mass value="0.8"/>
-      <inertia ixx="0.01" ixy="0.0" ixz="0.0" iyy="0.01" iyz="0.0" izz="0.005"/>
+      <origin xyz="0 0 0" rpy="0 0 0"/>
+      <geometry>
+        <mesh filename="file:///home/juptegraph/Workspaces/Robotics/Projects/CORI/cori_ws/src/cori_description/meshes/cori_body_v1.0/cori_left_upper_arm.stl" scale="0.35 0.35 0.35"/>
+      </geometry>
+      <material name="cori_white"/>
+    </visual>
+    <collision>
+      <geometry>
+        <box size="0.05 0.07 0.13"/>
+      </geometry>
+    </collision>
+    <inertial>
+      <mass value="0.9"/>
+      <origin xyz="0 0 -0.065"/>
+      <inertia ixx="0.015" ixy="0.0" ixz="0.0" iyy="0.015" iyz="0.0" izz="0.008"/>
     </inertial>
   </link>
@@ -104,21 +116,24 @@
     <parent link="torso"/>
     <child link="left_upper_arm"/>
-    <origin xyz="0 0 0" rpy="0 0 0"/>
+    <!-- Active Testing  -->
+    <origin xyz="-0.07 0 0" rpy="0 0.15 0"/>  <!-- Zero distance -->
   </joint>
   <link name="left_forearm">
     <visual>
-      <geometry>
-        <mesh filename="file:///home/juptegraph/Workspaces/Robotics/Projects/CORI/cori_ws/src/cori_description/meshes/cori_body_v1.0/cori_left_forearm.stl" scale="0.4 0.4 0.4"/>
-      </geometry>
-      <material name="cori_material"/>
-    </visual>
-    <collision>
-      <geometry>
-        <mesh filename="file:///home/juptegraph/Workspaces/Robotics/Projects/CORI/cori_ws/src/cori_description/meshes/cori_body_v1.0/cori_left_forearm.stl" scale="0.4 0.4 0.4"/>
-      </geometry>
-    </collision>
-    <inertial>
-      <mass value="0.6"/>
-      <inertia ixx="0.008" ixy="0.0" ixz="0.0" iyy="0.008" iyz="0.0" izz="0.004"/>
+      <origin xyz="0 0 0" rpy="0 0 0"/>
+      <geometry>
+        <mesh filename="file:///home/juptegraph/Workspaces/Robotics/Projects/CORI/cori_ws/src/cori_description/meshes/cori_body_v1.0/cori_left_forearm.stl" scale="0.35 0.35 0.35"/>
+      </geometry>
+      <material name="cori_white"/>
+    </visual>
+    <collision>
+      <geometry>
+        <box size="0.04 0.06 0.11"/>
+      </geometry>
+    </collision>
+    <inertial>
+      <mass value="0.55"/>
+      <origin xyz="0 0 -0.055"/>
+      <inertia ixx="0.012" ixy="0.0" ixz="0.0" iyy="0.012" iyz="0.0" izz="0.006"/>
     </inertial>
   </link>
@@ -126,21 +141,23 @@
     <parent link="left_upper_arm"/>
     <child link="left_forearm"/>
-    <origin xyz="0 0 0" rpy="0 0 0"/>
+    <origin xyz="0 0 0" rpy="0 0 0"/>  <!-- Zero distance -->
   </joint>
   <link name="left_hand">
     <visual>
-      <geometry>
-        <mesh filename="file:///home/juptegraph/Workspaces/Robotics/Projects/CORI/cori_ws/src/cori_description/meshes/cori_body_v1.0/cori_left_hand.stl" scale="0.4 0.4 0.4"/>
-      </geometry>
-      <material name="cori_material"/>
-    </visual>
-    <collision>
-      <geometry>
-        <mesh filename="file:///home/juptegraph/Workspaces/Robotics/Projects/CORI/cori_ws/src/cori_description/meshes/cori_body_v1.0/cori_left_hand.stl" scale="0.4 0.4 0.4"/>
-      </geometry>
-    </collision>
-    <inertial>
-      <mass value="0.3"/>
-      <inertia ixx="0.005" ixy="0.0" ixz="0.0" iyy="0.005" iyz="0.0" izz="0.005"/>
+      <origin xyz="0 0 0" rpy="0 0 0"/>
+      <geometry>
+        <mesh filename="file:///home/juptegraph/Workspaces/Robotics/Projects/CORI/cori_ws/src/cori_description/meshes/cori_body_v1.0/cori_left_hand.stl" scale="0.35 0.35 0.35"/>
+      </geometry>
+      <material name="cori_white"/>
+    </visual>
+    <collision>
+      <geometry>
+        <box size="0.05 0.035 0.07"/>
+      </geometry>
+    </collision>
+    <inertial>
+      <mass value="0.25"/>
+      <origin xyz="0 0 0"/>
+      <inertia ixx="0.008" ixy="0.0" ixz="0.0" iyy="0.008" iyz="0.0" izz="0.008"/>
     </inertial>
   </link>
@@ -148,22 +165,23 @@
     <parent link="left_forearm"/>
     <child link="left_hand"/>
-    <origin xyz="0 0 0" rpy="0 0 0"/>
-  </joint>
-  <!-- RIGHT ARM ASSEMBLY -->
+    <origin xyz="0 0 0" rpy="0 0 0"/>  <!-- Zero distance -->
+  </joint>
   <link name="right_upper_arm">
     <visual>
-      <geometry>
-        <mesh filename="file:///home/juptegraph/Workspaces/Robotics/Projects/CORI/cori_ws/src/cori_description/meshes/cori_body_v1.0/cori_right_upper_arm.stl" scale="0.4 0.4 0.4"/>
-      </geometry>
-      <material name="cori_material"/>
-    </visual>
-    <collision>
-      <geometry>
-        <mesh filename="file:///home/juptegraph/Workspaces/Robotics/Projects/CORI/cori_ws/src/cori_description/meshes/cori_body_v1.0/cori_right_upper_arm.stl" scale="0.4 0.4 0.4"/>
-      </geometry>
-    </collision>
-    <inertial>
-      <mass value="0.8"/>
-      <inertia ixx="0.01" ixy="0.0" ixz="0.0" iyy="0.01" iyz="0.0" izz="0.005"/>
+      <origin xyz="0 0 0" rpy="0 0 0"/>
+      <geometry>
+        <mesh filename="file:///home/juptegraph/Workspaces/Robotics/Projects/CORI/cori_ws/src/cori_description/meshes/cori_body_v1.0/cori_right_upper_arm.stl" scale="0.35 0.35 0.35"/>
+      </geometry>
+      <material name="cori_white"/>
+    </visual>
+    <collision>
+      <geometry>
+        <box size="0.05 0.07 0.13"/>
+      </geometry>
+    </collision>
+    <inertial>
+      <mass value="0.9"/>
+      <origin xyz="0 0 -0.065"/>
+      <inertia ixx="0.015" ixy="0.0" ixz="0.0" iyy="0.0" iyz="0.0" izz="0.00"/>
     </inertial>
   </link>
@@ -171,21 +189,24 @@
     <parent link="torso"/>
     <child link="right_upper_arm"/>
-    <origin xyz="0 0 0" rpy="0 0 0"/>
+    <!-- Actively Testing -->
+    <origin xyz="0.07 0 0" rpy="0 -0.15 0"/>  <!-- Zero distance -->
   </joint>
   <link name="right_forearm">
     <visual>
-      <geometry>
-        <mesh filename="file:///home/juptegraph/Workspaces/Robotics/Projects/CORI/cori_ws/src/cori_description/meshes/cori_body_v1.0/cori_right_forearm.stl" scale="0.4 0.4 0.4"/>
-      </geometry>
-      <material name="cori_material"/>
-    </visual>
-    <collision>
-      <geometry>
-        <mesh filename="file:///home/juptegraph/Workspaces/Robotics/Projects/CORI/cori_ws/src/cori_description/meshes/cori_body_v1.0/cori_right_forearm.stl" scale="0.4 0.4 0.4"/>
-      </geometry>
-    </collision>
-    <inertial>
-      <mass value="0.6"/>
-      <inertia ixx="0.008" ixy="0.0" ixz="0.0" iyy="0.008" iyz="0.0" izz="0.004"/>
+      <origin xyz="0 0 0" rpy="0 0 0"/>
+      <geometry>
+        <mesh filename="file:///home/juptegraph/Workspaces/Robotics/Projects/CORI/cori_ws/src/cori_description/meshes/cori_body_v1.0/cori_right_forearm.stl" scale="0.35 0.35 0.35"/>
+      </geometry>
+      <material name="cori_white"/>
+    </visual>
+    <collision>
+      <geometry>
+        <box size="0.04 0.06 0.11"/>
+      </geometry>
+    </collision>
+    <inertial>
+      <mass value="0.55"/>
+      <origin xyz="0 0 -0.055"/>
+      <inertia ixx="0.012" ixy="0.0" ixz="0.0" iyy="0.012" iyz="0.0" izz="0.006"/>
     </inertial>
   </link>
@@ -193,21 +214,23 @@
     <parent link="right_upper_arm"/>
     <child link="right_forearm"/>
-    <origin xyz="0 0 0" rpy="0 0 0"/>
+    <origin xyz="0 0 0" rpy="0 0 0"/>  <!-- Zero distance -->
   </joint>
   <link name="right_hand">
     <visual>
-      <geometry>
-        <mesh filename="file:///home/juptegraph/Workspaces/Robotics/Projects/CORI/cori_ws/src/cori_description/meshes/cori_body_v1.0/cori_right_hand.stl" scale="0.4 0.4 0.4"/>
-      </geometry>
-      <material name="cori_material"/>
-    </visual>
-    <collision>
-      <geometry>
-        <mesh filename="file:///home/juptegraph/Workspaces/Robotics/Projects/CORI/cori_ws/src/cori_description/meshes/cori_body_v1.0/cori_right_hand.stl" scale="0.4 0.4 0.4"/>
-      </geometry>
-    </collision>
-    <inertial>
-      <mass value="0.3"/>
-      <inertia ixx="0.005" ixy="0.0" ixz="0.0" iyy="0.005" iyz="0.0" izz="0.005"/>
+      <origin xyz="0 0 0" rpy="0 0 0"/>
+      <geometry>
+        <mesh filename="file:///home/juptegraph/Workspaces/Robotics/Projects/CORI/cori_ws/src/cori_description/meshes/cori_body_v1.0/cori_right_hand.stl" scale="0.35 0.35 0.35"/>
+      </geometry>
+      <material name="cori_white"/>
+    </visual>
+    <collision>
+      <geometry>
+        <box size="0.05 0.035 0.07"/>
+      </geometry>
+    </collision>
+    <inertial>
+      <mass value="0.25"/>
+      <origin xyz="0 0 0"/>
+      <inertia ixx="0.008" ixy="0.0" ixz="0.0" iyy="0.008" iyz="0.0" izz="0.008"/>
     </inertial>
   </link>
@@ -215,44 +238,47 @@
     <parent link="right_forearm"/>
     <child link="right_hand"/>
-    <origin xyz="0 0 0" rpy="0 0 0"/>
-  </joint>
-  <!-- LEFT LEG ASSEMBLY -->
+    <origin xyz="0 0 0" rpy="0 0 0"/>  <!-- Zero distance -->
+  </joint>
   <link name="left_thigh">
     <visual>
-      <geometry>
-        <mesh filename="file:///home/juptegraph/Workspaces/Robotics/Projects/CORI/cori_ws/src/cori_description/meshes/cori_body_v1.0/cori_left_thigh.stl" scale="0.4 0.4 0.4"/>
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
Commit message: Documented and attempted to fix neck rotation issues... still unresolved... will attempt tomorrow AM.

File: cori_ws/install/cori_description/share/cori_description/urdf/cori.urdf.xacro (robot description, xacro)
@@ -59,5 +59,5 @@
       <mass value="1.8"/>
       <origin xyz="0 0 0"/>
-      <inertia ixx="0.018" ixy="0.0" ixz="0.0" iyy="0.0" iyz="0.0" izz="0.018"/>
+      <inertia ixx="0.018" ixy="0.0" ixz="0.0" iyy="0.018" iyz="0.0" izz="0.018"/>
     </inertial>
   </link>

File: cori_ws/src/cori_description/urdf/cori.urdf.xacro (robot description, xacro)
@@ -116,5 +116,5 @@
     <parent link="torso"/>
     <child link="left_upper_arm"/>
-    <!-- Active Testing  -->
+    <!-- Active Testing -->
     <origin xyz="-0.07 0 0" rpy="0 0.15 0"/>  <!-- Zero distance -->
   </joint>
