Commit message: First attempt at placing CORI full render in Gazebo

File: cori_ws/cori.urdf (robot description, URDF)
Before this commit: robot cori, 30 links, 29 joints
Links:
- removed link left_arm_wrist
- removed link left_finger_1
- removed link left_finger_2
- removed link left_finger_3
- removed link left_finger_4
- removed link left_leg_ankle
- removed link right_arm_wrist
- removed link right_leg_ankle
- added link full_body_collision; collision mesh filename=package://cori_description/meshes/CORI_Solid.stl scale=0.001 0.001 0.001
- link base_link: geometry collision cylinder length=0.02 radius=0.05; visual cylinder length=0.02 radius=0.05
- link head: geometry visual box size=0.28 0.2 0.14
- link left_arm_elbow: mass None -> 0.3; geometry collision cylinder length=0.04 radius=0.0225; visual cylinder length=0.04 radius=0.0225
- link left_arm_forearm: geometry visual cylinder length=0.26 radius=0.025
- link left_arm_upper: geometry visual cylinder length=0.28 radius=0.0275
- link left_eye: mass None -> 0.01
- link left_foot: geometry collision box size=0.24 0.12 0.045; visual box size=0.24 0.12 0.045
- link left_hand_palm: geometry collision box size=0.085 0.06 0.025; visual box size=0.085 0.06 0.025
- link left_leg_hip: geometry collision cylinder length=0.04 radius=0.03; visual cylinder length=0.04 radius=0.03
- link left_leg_shin: geometry visual cylinder length=0.32 radius=0.0275
- link left_leg_thigh: geometry visual cylinder length=0.35 radius=0.03
- link right_arm_elbow: mass None -> 0.3; geometry collision cylinder length=0.04 radius=0.0225; visual cylinder length=0.04 radius=0.0225
- link right_arm_forearm: geometry visual cylinder length=0.26 radius=0.025
- link right_arm_upper: geometry visual cylinder length=0.28 radius=0.0275
- link right_eye: mass None -> 0.01
- link right_foot: geometry collision box size=0.24 0.12 0.045; visual box size=0.24 0.12 0.045
- link right_hand_palm: geometry collision box size=0.085 0.06 0.025; visual box size=0.085 0.06 0.025
- link right_leg_hip: geometry collision cylinder length=0.04 radius=0.03; visual cylinder length=0.04 radius=0.03
- link right_leg_shin: geometry visual cylinder length=0.32 radius=0.0275
- link right_leg_thigh: geometry visual cylinder length=0.35 radius=0.03
- link screen: mass None -> 0.1; geometry visual box size=0.22 0.01 0.12
- link torso: geometry visual box size=0.32 0.22 0.38
Joints:
- removed joint left_ankle_end_joint
- removed joint left_finger_1_joint
- removed joint left_finger_2_joint
- removed joint left_finger_3_joint
- removed joint left_finger_4_joint
- removed joint left_wrist_end_joint
- removed joint right_ankle_end_joint
- removed joint right_wrist_end_joint
- added joint body_collision_joint: type fixed, parent base_link, child full_body_collision, origin xyz=0 0 0 rpy=0 0 0
- joint left_ankle_foot_joint: origin xyz=0 0 -0.045 rpy=0 0 0 -> xyz=0 0 -0.1825 rpy=0 0 0; parent left_leg_ankle -> left_leg_shin
- joint left_ankle_joint: limit lower=-2.09 upper=2.09 effort=100.0 velocity=1.0 -> (none); origin xyz=0 0 0.35 rpy=0 0 0 -> xyz=0 0 -0.175 rpy=0 0 0
- joint left_elbow_joint: limit lower=-2.09 upper=2.09 effort=100.0 velocity=1.0 -> (none); origin xyz=0 0 0.28 rpy=0 0 0 -> xyz=0 0 0.14 rpy=0 0 0
- joint left_eye_joint: origin (none) -> xyz=-0.08 0.02 0.02 rpy=0 0 0
- joint left_hip_joint: limit lower=-2.09 upper=2.09 effort=100.0 velocity=1.0 -> (none); origin xyz=-0.16 0 0 rpy=0 0 0 -> xyz=-0.08 0 -0.19 rpy=0 0 0
- joint left_knee_joint: limit lower=-2.09 upper=2.09 effort=100.0 velocity=1.0 -> (none); origin xyz=0 0 0.04 rpy=0 0 0 -> xyz=0 0 -0.175 rpy=0 0 0
- joint left_shoulder_joint: limit lower=-2.09 upper=2.09 effort=100.0 velocity=1.0 -> (none)
- joint left_wrist_hand_joint: origin xyz=0 0 0 rpy=0 0 0 -> xyz=0 0 0.13 rpy=0 0 0; parent left_arm_wrist -> left_arm_forearm
- joint left_wrist_joint: limit lower=-2.09 upper=2.09 effort=100.0 velocity=1.0 -> (none); origin xyz=0 0 0.04 rpy=0 0 0 -> xyz=0 0 0.02 rpy=0 0 0
- joint neck_joint: limit lower=-2.09 upper=2.09 effort=100.0 velocity=1.0 -> (none)
- joint right_ankle_foot_joint: origin xyz=0 0 -0.045 rpy=0 0 0 -> xyz=0 0 -0.1825 rpy=0 0 0; parent right_leg_ankle -> right_leg_shin
- joint right_ankle_joint: limit lower=-2.09 upper=2.09 effort=100.0 velocity=1.0 -> (none); origin xyz=0 0 0.35 rpy=0 0 0 -> xyz=0 0 -0.175 rpy=0 0 0
- joint right_elbow_joint: limit lower=-2.09 upper=2.09 effort=100.0 velocity=1.0 -> (none); origin xyz=0 0 0.28 rpy=0 0 0 -> xyz=0 0 0.14 rpy=0 0 0
- joint right_eye_joint: origin (none) -> xyz=0.08 0.02 0.02 rpy=0 0 0
- joint right_hip_joint: limit lower=-2.09 upper=2.09 effort=100.0 velocity=1.0 -> (none); origin xyz=0.16 0 0 rpy=0 0 0 -> xyz=0.08 0 -0.19 rpy=0 0 0
- joint right_knee_joint: limit lower=-2.09 upper=2.09 effort=100.0 velocity=1.0 -> (none); origin xyz=0 0 0.04 rpy=0 0 0 -> xyz=0 0 -0.175 rpy=0 0 0
- joint right_shoulder_joint: limit lower=-2.09 upper=2.09 effort=100.0 velocity=1.0 -> (none)
- joint right_wrist_hand_joint: origin xyz=0 0 0 rpy=0 0 0 -> xyz=0 0 0.13 rpy=0 0 0; parent right_arm_wrist -> right_arm_forearm
- joint right_wrist_joint: limit lower=-2.09 upper=2.09 effort=100.0 velocity=1.0 -> (none); origin xyz=0 0 0.04 rpy=0 0 0 -> xyz=0 0 0.02 rpy=0 0 0
- joint screen_joint: origin xyz=0 0 0.05 rpy=0 0 0 -> xyz=0 0.1 0.02 rpy=0 0 0
- joint waist_joint: limit lower=-2.09 upper=2.09 effort=100.0 velocity=1.0 -> (none)

File: cori_ws/src/cori_description/urdf/cori.urdf.xacro (robot description, xacro)
@@ -1,27 +1,152 @@
 <?xml version="1.0"?>
 <robot name="cori" xmlns:xacro="http://www.ros.org/wiki/xacro">
-  <!-- Materials -->
-  <material name="body_material">
-    <color rgba="0.82 0.81 0.78 1.0"/> <!-- Light gray for body -->
-  </material>
-  <material name="joint_material">
-    <color rgba="0.35 0.35 0.35 1.0"/> <!-- Dark gray for joints -->
-  </material>
-  <material name="screen_material">
-    <color rgba="0.05 0.05 0.05 1.0"/> <!-- Black for screen -->
-  </material>
-  <material name="eye_material">
-    <color rgba="1.0 1.0 1.0 1.0"/> <!-- White for eyes -->
-  </material>
-  <!-- Joint Properties Macro -->
-  <xacro:macro name="joint_properties">
-    <limit lower="-2.09" upper="2.09" effort="100.0" velocity="1.0"/>
-    <dynamics damping="0.7" friction="0.9"/>
-  </xacro:macro>
-  <!-- Base Link -->
-  <link name="base_link">
+<!-- Materials -->
+<material name="body_material">
+  <color rgba="0.82 0.81 0.78 1.0"/> <!-- Light gray for body -->
+</material>
+<material name="joint_material">
+  <color rgba="0.35 0.35 0.35 1.0"/> <!-- Dark gray for joints -->
+</material>
+<material name="screen_material">
+  <color rgba="0.05 0.05 0.05 1.0"/> <!-- Black for screen -->
+</material>
+<material name="eye_material">
+  <color rgba="1.0 1.0 1.0 1.0"/> <!-- White for eyes -->
+</material>
+<!-- Joint Properties Macro -->
+<xacro:macro name="joint_properties">
+  <limit lower="-2.09" upper="2.09" effort="100.0" velocity="1.0"/>
+  <dynamics damping="0.7" friction="0.9"/>
+</xacro:macro>
+<!-- Base Link -->
+<link name="base_link">
+  <visual>
+    <geometry>
+      <cylinder radius="0.05" length="0.02"/>
+    </geometry>
+    <material name="joint_material"/>
+  </visual>
+  <collision>
+    <geometry>
+      <cylinder radius="0.05" length="0.02"/>
+    </geometry>
+  </collision>
+  <inertial>
+    <mass value="0.1"/>
+    <inertia ixx="0.001" ixy="0.0" ixz="0.0" iyy="0.001" iyz="0.0" izz="0.001"/>
+  </inertial>
+</link>
+<!-- Full Body Collision Link using STL -->
+<link name="full_body_collision">
+  <collision>
+    <geometry>
+      <mesh filename="meshes/CORI_Solid.stl" scale="0.001 0.001 0.001"/>
+    </geometry>
+  </collision>
+</link>
+<joint name="body_collision_joint" type="fixed">
+  <parent link="base_link"/>
+  <child link="full_body_collision"/>
+  <origin xyz="0 0 0" rpy="0 0 0"/>
+</joint>
+<!-- Head Assembly -->
+<link name="head">
+  <visual>
+    <geometry>
+      <box size="0.28 0.2 0.14"/>
+    </geometry>
+    <material name="body_material"/>
+  </visual>
+  <!-- Removed individual collision - using full body STL instead -->
+  <inertial>
+    <mass value="1.5"/>
+    <inertia ixx="0.015" ixy="0.0" ixz="0.0" iyy="0.015" iyz="0.0" izz="0.015"/>
+  </inertial>
+</link>
+<joint name="neck_joint" type="revolute">
+  <parent link="base_link"/>
+  <child link="head"/>
+  <axis xyz="0 0 1"/>
+  <xacro:joint_properties/>
+  <origin xyz="0 0 0.38" rpy="0 0 0"/>
+</joint>
+<link name="screen">
+  <visual>
+    <geometry>
+      <box size="0.22 0.01 0.12"/>
+    </geometry>
+    <material name="screen_material"/>
+  </visual>
+  <inertial>
+    <mass value="0.1"/>
+    <inertia ixx="0.001" ixy="0.0" ixz="0.0" iyy="0.001" iyz="0.0" izz="0.001"/>
+  </inertial>
+</link>
+<joint name="screen_joint" type="fixed">
+  <parent link="head"/>
+  <child link="screen"/>
+  <origin xyz="0 0.1 0.02" rpy="0 0 0"/>
+</joint>
+<link name="left_eye">
+  <visual>
+    <geometry>
+      <sphere radius="0.015"/>
+    </geometry>
+    <material name="eye_material"/>
+  </visual>
+  <inertial>
+    <mass value="0.01"/>
+    <inertia ixx="0.0001" ixy="0.0" ixz="0.0" iyy="0.0001" iyz="0.0" izz="0.0001"/>
+  </inertial>
+</link>
+<joint name="left_eye_joint" type="fixed">
+  <parent link="screen"/>
+  <child link="left_eye"/>
+  <origin xyz="-0.08 0.02 0.02" rpy="0 0 0"/>
+</joint>
+<link name="right_eye">
+  <visual>
+    <geometry>
+      <sphere radius="0.015"/>
+    </geometry>
+    <material name="eye_material"/>
+  </visual>
+  <inertial>
+    <mass value="0.01"/>
+    <inertia ixx="0.0001" ixy="0.0" ixz="0.0" iyy="0.0001" iyz="0.0" izz="0.0001"/>
+  </inertial>
+</link>
+<joint name="right_eye_joint" type="fixed">
+  <parent link="screen"/>
+  <child link="right_eye"/>
+  <origin xyz="0.08 0.02 0.02" rpy="0 0 0"/>
+</joint>
+<!-- Torso Assembly -->
+<link name="torso">
+  <visual>
+    <geometry>
+      <box size="0.32 0.22 0.38"/>
+    </geometry>
+    <material name="body_material"/>
+  </visual>
+  <!-- Removed individual collision - using full body STL instead -->
+  <inertial>
+    <mass value="8.0"/>
+    <inertia ixx="0.08" ixy="0.0" ixz="0.0" iyy="0.08" iyz="0.0" izz="0.08"/>
+  </inertial>
+</link>
+<joint name="waist_joint" type="revolute">
+  <parent link="base_link"/>
+  <child link="torso"/>
+  <axis xyz="0 0 1"/>
+  <xacro:joint_properties/>
+  <origin xyz="0 0 0" rpy="0 0 0"/>
+</joint>
+<!-- Finger Macro -->
+<xacro:macro name="finger" params="hand name offset">
+  <link name="${hand}_finger_${name}">
     <visual>
       <geometry>
-        <cylinder radius="0.05" length="0.02"/>
+        <cylinder radius="0.006" length="0.06"/>
       </geometry>
       <material name="joint_material"/>
@@ -29,550 +154,383 @@
     <collision>
       <geometry>
-        <cylinder radius="0.05" length="0.02"/>
+        <cylinder radius="0.006" length="0.06"/>
       </geometry>
     </collision>
     <inertial>
       <mass value="0.1"/>
-      <inertia ixx="0.001" ixy="0.0" ixz="0.0" iyy="0.001" iyz="0.0" izz="0.001"/>
-    </inertial>
-  </link>
-  <!-- Head Assembly -->
-  <link name="head">
-    <visual>
-      <geometry>
-        <box size="0.28 0.2 0.14"/>
-      </geometry>
-      <material name="body_material"/>
-    </visual>
-    <collision>
-      <geometry>
-        <box size="0.28 0.2 0.14"/>
-      </geometry>
-    </collision>
-    <inertial>
-      <mass value="1.5"/>
-      <inertia ixx="0.015" ixy="0.0" ixz="0.0" iyy="0.015" iyz="0.0" izz="0.015"/>
-    </inertial>
-  </link>
-  <joint name="neck_joint" type="revolute">
-    <parent link="base_link"/>
-    <child link="head"/>
-    <axis xyz="0 0 1"/>
-    <xacro:joint_properties/>
-    <origin xyz="0 0 0.38" rpy="0 0 0"/>
-  </joint>
-  <link name="screen">
-    <visual>
-      <geometry>
-        <box size="0.22 0.01 0.12"/>
-      </geometry>
-      <material name="screen_material"/>
-    </visual>
-    <collision>
-      <geometry>
-        <box size="0.22 0.01 0.12"/>
-      </geometry>
-    </collision>
-    <inertial>
-      <mass value="0.1"/>
-      <inertia ixx="0.001" ixy="0.0" ixz="0.0" iyy="0.001" iyz="0.0" izz="0.001"/>
-    </inertial>
-  </link>
-  <joint name="screen_joint" type="fixed">
-    <parent link="head"/>
-    <child link="screen"/>
-    <origin xyz="0 0.1 0.02" rpy="0 0 0"/>
-  </joint>
-  <link name="left_eye">
-    <visual>
-      <geometry>
-        <sphere radius="0.015"/>
-      </geometry>
-      <material name="eye_material"/>
-    </visual>
-    <collision>
-      <geometry>
-        <sphere radius="0.015"/>
-      </geometry>
-    </collision>
-    <inertial>
-      <mass value="0.01"/>
       <inertia ixx="0.0001" ixy="0.0" ixz="0.0" iyy="0.0001" iyz="0.0" izz="0.0001"/>
     </inertial>
   </link>
-  <joint name="left_eye_joint" type="fixed">
-    <parent link="screen"/>
-    <child link="left_eye"/>
-    <origin xyz="-0.08 0.02 0.02" rpy="0 0 0"/>
+  <joint name="${hand}_finger_${name}_joint" type="revolute">
+    <parent link="${hand}_hand_palm"/>
+    <child link="${hand}_finger_${name}"/>
+    <axis xyz="0 0 1"/>
+    <limit lower="0.0" upper="1.57" effort="50.0" velocity="0.5"/>
+    <dynamics damping="0.5" friction="0.7"/>
+    <origin xyz="${offset} 0 -0.025" rpy="0 0 0"/>
   </joint>
-  <link name="right_eye">
-    <visual>
-      <geometry>
-        <sphere radius="0.015"/>
-      </geometry>
-      <material name="eye_material"/>
-    </visual>
-    <collision>
-      <geometry>
-        <sphere radius="0.015"/>
-      </geometry>
-    </collision>
-    <inertial>
-      <mass value="0.01"/>
-      <inertia ixx="0.0001" ixy="0.0" ixz="0.0" iyy="0.0001" iyz="0.0" izz="0.0001"/>
-    </inertial>
-  </link>
-  <joint name="right_eye_joint" type="fixed">
-    <parent link="screen"/>
-    <child link="right_eye"/>
-    <origin xyz="0.08 0.02 0.02" rpy="0 0 0"/>
-  </joint>
-  <!-- Torso Assembly -->
-  <link name="torso">
-    <visual>
-      <geometry>
-        <box size="0.32 0.22 0.38"/>
-      </geometry>
-      <material name="body_material"/>
-    </visual>
-    <collision>
-      <geometry>
-        <box size="0.32 0.22 0.38"/>
-      </geometry>
-    </collision>
-    <inertial>
-      <mass value="8.0"/>
-      <inertia ixx="0.08" ixy="0.0" ixz="0.0" iyy="0.08" iyz="0.0" izz="0.08"/>
-    </inertial>
-  </link>
-  <joint name="waist_joint" type="revolute">
-    <parent link="base_link"/>
-    <child link="torso"/>
-    <axis xyz="0 0 1"/>
-    <xacro:joint_properties/>
-    <origin xyz="0 0 0" rpy="0 0 0"/>
-  </joint>
-  <!-- Finger Macro -->
-  <xacro:macro name="finger" params="hand name offset">
-    <link name="${hand}_finger_${name}">
-      <visual>
-        <geometry>
-          <cylinder radius="0.006" length="0.06"/>
-        </geometry>
-        <material name="joint_material"/>
-      </visual>
-      <collision>
-        <geometry>
-          <cylinder radius="0.006" length="0.06"/>
-        </geometry>
-      </collision>
-      <inertial>
-        <mass value="0.1"/>
-        <inertia ixx="0.0001" ixy="0.0" ixz="0.0" iyy="0.0001" iyz="0.0" izz="0.0001"/>
-      </inertial>
-    </link>
-    <joint name="${hand}_finger_${name}_joint" type="revolute">
-      <parent link="${hand}_hand_palm"/>
-      <child link="${hand}_finger_${name}"/>
-      <axis xyz="0 0 1"/>
-      <limit lower="0.0" upper="1.57" effort="50.0" velocity="0.5"/>
-      <dynamics damping="0.5" friction="0.7"/>
-      <origin xyz="${offset} 0 -0.025" rpy="0 0 0"/>
-    </joint>
-  </xacro:macro>
-  <!-- Left Arm -->
-  <link name="left_arm_upper">
-    <visual>
-      <geometry>
-        <cylinder radius="0.0275" length="0.28"/>
-      </geometry>
-      <material name="body_material"/>
-    </visual>
-    <collision>
-      <geometry>
-        <cylinder radius="0.0275" length="0.28"/>
-      </geometry>
-    </collision>
-    <inertial>
-      <mass value="1.2"/>
-      <inertia ixx="0.012" ixy="0.0" ixz="0.0" iyy="0.012" iyz="0.0" izz="0.012"/>
-    </inertial>
-  </link>
-  <joint name="left_shoulder_joint" type="revolute">
-    <parent link="torso"/>
-    <child link="left_arm_upper"/>
-    <axis xyz="0 1 0"/>
-    <xacro:joint_properties/>
-    <origin xyz="-0.16 0 0.38" rpy="0 0 0"/>
-  </joint>
-  <link name="left_arm_elbow">
-    <visual>
-      <geometry>
-        <cylinder radius="0.0225" length="0.04"/>
-      </geometry>
-      <material name="joint_material"/>
-    </visual>
-    <collision>
-      <geometry>
-        <cylinder radius="0.0225" length="0.04"/>
-      </geometry>
-    </collision>
-    <inertial>
-      <mass value="0.3"/>
-      <inertia ixx="0.003" ixy="0.0" ixz="0.0" iyy="0.003" iyz="0.0" izz="0.003"/>
-    </inertial>
-  </link>
-  <joint name="left_elbow_joint" type="revolute">
-    <parent link="left_arm_upper"/>
-    <child link="left_arm_elbow"/>
-    <axis xyz="0 1 0"/>
-    <xacro:joint_properties/>
-    <origin xyz="0 0 0.14" rpy="0 0 0"/>
-  </joint>
-  <link name="left_arm_forearm">
-    <visual>
-      <geometry>
-        <cylinder radius="0.025" length="0.26"/>
-      </geometry>
-      <material name="body_material"/>
-    </visual>
-    <collision>
-      <geometry>
-        <cylinder radius="0.025" length="0.26"/>
-      </geometry>
-    </collision>
-    <inertial>
-      <mass value="1.0"/>
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