Commit message: Began Gazebo Configuration for CORI

File: cori_ws/src/cori_description/urdf/cori.urdf.xacro (robot description, xacro)
@@ -1,122 +1,578 @@
 <?xml version="1.0"?>
-<robot name="cori_robot">
-  <material name="light_grey">
-    <color rgba="0.8 0.8 0.8 1.0"/>
+<robot name="cori" xmlns:xacro="http://www.ros.org/wiki/xacro">
+  <!-- Materials -->
+  <material name="body_material">
+    <color rgba="0.82 0.81 0.78 1.0"/> <!-- Light gray for body -->
   </material>
-  <material name="dark_grey">
-    <color rgba="0.4 0.4 0.4 1.0"/>
+  <material name="joint_material">
+    <color rgba="0.35 0.35 0.35 1.0"/> <!-- Dark gray for joints -->
   </material>
+  <material name="screen_material">
+    <color rgba="0.05 0.05 0.05 1.0"/> <!-- Black for screen -->
+  </material>
+  <material name="eye_material">
+    <color rgba="1.0 1.0 1.0 1.0"/> <!-- White for eyes -->
+  </material>
+  <!-- Joint Properties Macro -->
+  <xacro:macro name="joint_properties">
+    <limit lower="-2.09" upper="2.09" effort="100.0" velocity="1.0"/>
+    <dynamics damping="0.7" friction="0.9"/>
+  </xacro:macro>
+  <!-- Base Link -->
   <link name="base_link">
     <visual>
-      <origin xyz="0 0 0" rpy="0 0 0"/>
-      <geometry>
-        <box size="0.25 0.18 0.35"/>
-      </geometry>
-      <material name="light_grey"/>
-    </visual>
-    <collision>
-      <origin xyz="0 0 0" rpy="0 0 0"/>
-      <geometry>
-        <box size="0.25 0.18 0.35"/>
-      </geometry>
-    </collision>
-    <inertial>
-      <origin xyz="0 0 0" rpy="0 0 0"/>
-      <mass value="8.5"/>
-      <inertia ixx="0.2" ixy="0" ixz="0" iyy="0.3" iyz="0" izz="0.15"/>
-    </inertial>
-  </link>
-  <link name="head_link">
-    <visual>
-      <origin xyz="0 0 0" rpy="0 0 0"/>
-      <geometry>
-        <box size="0.20 0.12 0.08"/>
-      </geometry>
-      <material name="light_grey"/>
-    </visual>
-    <collision>
-      <origin xyz="0 0 0" rpy="0 0 0"/>
-      <geometry>
-        <box size="0.20 0.12 0.08"/>
-      </geometry>
-    </collision>
-    <inertial>
-      <origin xyz="0 0 0" rpy="0 0 0"/>
+      <geometry>
+        <cylinder radius="0.05" length="0.02"/>
+      </geometry>
+      <material name="joint_material"/>
+    </visual>
+    <collision>
+      <geometry>
+        <cylinder radius="0.05" length="0.02"/>
+      </geometry>
+    </collision>
+    <inertial>
+      <mass value="0.1"/>
+      <inertia ixx="0.001" ixy="0.0" ixz="0.0" iyy="0.001" iyz="0.0" izz="0.001"/>
+    </inertial>
+  </link>
+  <!-- Head Assembly -->
+  <link name="head">
+    <visual>
+      <geometry>
+        <box size="0.28 0.2 0.14"/>
+      </geometry>
+      <material name="body_material"/>
+    </visual>
+    <collision>
+      <geometry>
+        <box size="0.28 0.2 0.14"/>
+      </geometry>
+    </collision>
+    <inertial>
+      <mass value="1.5"/>
+      <inertia ixx="0.015" ixy="0.0" ixz="0.0" iyy="0.015" iyz="0.0" izz="0.015"/>
+    </inertial>
+  </link>
+  <joint name="neck_joint" type="revolute">
+    <parent link="base_link"/>
+    <child link="head"/>
+    <axis xyz="0 0 1"/>
+    <xacro:joint_properties/>
+    <origin xyz="0 0 0.38" rpy="0 0 0"/>
+  </joint>
+  <link name="screen">
+    <visual>
+      <geometry>
+        <box size="0.22 0.01 0.12"/>
+      </geometry>
+      <material name="screen_material"/>
+    </visual>
+    <collision>
+      <geometry>
+        <box size="0.22 0.01 0.12"/>
+      </geometry>
+    </collision>
+    <inertial>
+      <mass value="0.1"/>
+      <inertia ixx="0.001" ixy="0.0" ixz="0.0" iyy="0.001" iyz="0.0" izz="0.001"/>
+    </inertial>
+  </link>
+  <joint name="screen_joint" type="fixed">
+    <parent link="head"/>
+    <child link="screen"/>
+    <origin xyz="0 0.1 0.02" rpy="0 0 0"/>
+  </joint>
+  <link name="left_eye">
+    <visual>
+      <geometry>
+        <sphere radius="0.015"/>
+      </geometry>
+      <material name="eye_material"/>
+    </visual>
+    <collision>
+      <geometry>
+        <sphere radius="0.015"/>
+      </geometry>
+    </collision>
+    <inertial>
+      <mass value="0.01"/>
+      <inertia ixx="0.0001" ixy="0.0" ixz="0.0" iyy="0.0001" iyz="0.0" izz="0.0001"/>
+    </inertial>
+  </link>
+  <joint name="left_eye_joint" type="fixed">
+    <parent link="screen"/>
+    <child link="left_eye"/>
+    <origin xyz="-0.08 0.02 0.02" rpy="0 0 0"/>
+  </joint>
+  <link name="right_eye">
+    <visual>
+      <geometry>
+        <sphere radius="0.015"/>
+      </geometry>
+      <material name="eye_material"/>
+    </visual>
+    <collision>
+      <geometry>
+        <sphere radius="0.015"/>
+      </geometry>
+    </collision>
+    <inertial>
+      <mass value="0.01"/>
+      <inertia ixx="0.0001" ixy="0.0" ixz="0.0" iyy="0.0001" iyz="0.0" izz="0.0001"/>
+    </inertial>
+  </link>
+  <joint name="right_eye_joint" type="fixed">
+    <parent link="screen"/>
+    <child link="right_eye"/>
+    <origin xyz="0.08 0.02 0.02" rpy="0 0 0"/>
+  </joint>
+  <!-- Torso Assembly -->
+  <link name="torso">
+    <visual>
+      <geometry>
+        <box size="0.32 0.22 0.38"/>
+      </geometry>
+      <material name="body_material"/>
+    </visual>
+    <collision>
+      <geometry>
+        <box size="0.32 0.22 0.38"/>
+      </geometry>
+    </collision>
+    <inertial>
+      <mass value="8.0"/>
+      <inertia ixx="0.08" ixy="0.0" ixz="0.0" iyy="0.08" iyz="0.0" izz="0.08"/>
+    </inertial>
+  </link>
+  <joint name="waist_joint" type="revolute">
+    <parent link="base_link"/>
+    <child link="torso"/>
+    <axis xyz="0 0 1"/>
+    <xacro:joint_properties/>
+    <origin xyz="0 0 0" rpy="0 0 0"/>
+  </joint>
+  <!-- Finger Macro -->
+  <xacro:macro name="finger" params="hand name offset">
+    <link name="${hand}_finger_${name}">
+      <visual>
+        <geometry>
+          <cylinder radius="0.006" length="0.06"/>
+        </geometry>
+        <material name="joint_material"/>
+      </visual>
+      <collision>
+        <geometry>
+          <cylinder radius="0.006" length="0.06"/>
+        </geometry>
+      </collision>
+      <inertial>
+        <mass value="0.1"/>
+        <inertia ixx="0.0001" ixy="0.0" ixz="0.0" iyy="0.0001" iyz="0.0" izz="0.0001"/>
+      </inertial>
+    </link>
+    <joint name="${hand}_finger_${name}_joint" type="revolute">
+      <parent link="${hand}_hand_palm"/>
+      <child link="${hand}_finger_${name}"/>
+      <axis xyz="0 0 1"/>
+      <limit lower="0.0" upper="1.57" effort="50.0" velocity="0.5"/>
+      <dynamics damping="0.5" friction="0.7"/>
+      <origin xyz="${offset} 0 -0.025" rpy="0 0 0"/>
+    </joint>
+  </xacro:macro>
+  <!-- Left Arm -->
+  <link name="left_arm_upper">
+    <visual>
+      <geometry>
+        <cylinder radius="0.0275" length="0.28"/>
+      </geometry>
+      <material name="body_material"/>
+    </visual>
+    <collision>
+      <geometry>
+        <cylinder radius="0.0275" length="0.28"/>
+      </geometry>
+    </collision>
+    <inertial>
       <mass value="1.2"/>
-      <inertia ixx="0.01" ixy="0" ixz="0" iyy="0.015" iyz="0" izz="0.02"/>
-    </inertial>
-  </link>
-  <joint name="head_joint" type="revolute">
-    <parent link="base_link"/>
-    <child link="head_link"/>
-    <origin xyz="0 0 0.22" rpy="0 0 0"/>
-    <axis xyz="0 0 1"/>
-    <limit lower="-1.57" upper="1.57" effort="50" velocity="2.0"/>
-  </joint>
-  <link name="left_shoulder_link">
-    <visual>
-      <origin xyz="0 0 0" rpy="0 0 0"/>
-      <geometry>
-        <cylinder radius="0.04" length="0.08"/>
-      </geometry>
-      <material name="dark_grey"/>
-    </visual>
-    <collision>
-      <origin xyz="0 0 0" rpy="0 0 0"/>
-      <geometry>
-        <cylinder radius="0.04" length="0.08"/>
-      </geometry>
-    </collision>
-    <inertial>
-      <origin xyz="0 0 0" rpy="0 0 0"/>
+      <inertia ixx="0.012" ixy="0.0" ixz="0.0" iyy="0.012" iyz="0.0" izz="0.012"/>
+    </inertial>
+  </link>
+  <joint name="left_shoulder_joint" type="revolute">
+    <parent link="torso"/>
+    <child link="left_arm_upper"/>
+    <axis xyz="0 1 0"/>
+    <xacro:joint_properties/>
+    <origin xyz="-0.16 0 0.38" rpy="0 0 0"/>
+  </joint>
+  <link name="left_arm_elbow">
+    <visual>
+      <geometry>
+        <cylinder radius="0.0225" length="0.04"/>
+      </geometry>
+      <material name="joint_material"/>
+    </visual>
+    <collision>
+      <geometry>
+        <cylinder radius="0.0225" length="0.04"/>
+      </geometry>
+    </collision>
+    <inertial>
+      <mass value="0.3"/>
+      <inertia ixx="0.003" ixy="0.0" ixz="0.0" iyy="0.003" iyz="0.0" izz="0.003"/>
+    </inertial>
+  </link>
+  <joint name="left_elbow_joint" type="revolute">
+    <parent link="left_arm_upper"/>
+    <child link="left_arm_elbow"/>
+    <axis xyz="0 1 0"/>
+    <xacro:joint_properties/>
+    <origin xyz="0 0 0.14" rpy="0 0 0"/>
+  </joint>
+  <link name="left_arm_forearm">
+    <visual>
+      <geometry>
+        <cylinder radius="0.025" length="0.26"/>
+      </geometry>
+      <material name="body_material"/>
+    </visual>
+    <collision>
+      <geometry>
+        <cylinder radius="0.025" length="0.26"/>
+      </geometry>
+    </collision>
+    <inertial>
+      <mass value="1.0"/>
+      <inertia ixx="0.01" ixy="0.0" ixz="0.0" iyy="0.01" iyz="0.0" izz="0.01"/>
+    </inertial>
+  </link>
+  <joint name="left_wrist_joint" type="revolute">
+    <parent link="left_arm_elbow"/>
+    <child link="left_arm_forearm"/>
+    <axis xyz="0 1 0"/>
+    <xacro:joint_properties/>
+    <origin xyz="0 0 0.02" rpy="0 0 0"/>
+  </joint>
+  <link name="left_hand_palm">
+    <visual>
+      <geometry>
+        <box size="0.085 0.06 0.025"/>
+      </geometry>
+      <material name="joint_material"/>
+    </visual>
+    <collision>
+      <geometry>
+        <box size="0.085 0.06 0.025"/>
+      </geometry>
+    </collision>
+    <inertial>
+      <mass value="0.6"/>
+      <inertia ixx="0.0015" ixy="0.0" ixz="0.0" iyy="0.0015" iyz="0.0" izz="0.0015"/>
+    </inertial>
+  </link>
+  <joint name="left_wrist_hand_joint" type="fixed">
+    <parent link="left_arm_forearm"/>
+    <child link="left_hand_palm"/>
+    <origin xyz="0 0 0.13" rpy="0 0 0"/>
+  </joint>
+  <!-- Left Hand Fingers -->
+  <xacro:finger hand="left" name="1" offset="-0.02"/>
+  <xacro:finger hand="left" name="2" offset="-0.0067"/>
+  <xacro:finger hand="left" name="3" offset="0.0067"/>
+  <xacro:finger hand="left" name="4" offset="0.02"/>
+  <!-- Right Arm (Mirrored) -->
+  <link name="right_arm_upper">
+    <visual>
+      <geometry>
+        <cylinder radius="0.0275" length="0.28"/>
+      </geometry>
+      <material name="body_material"/>
+    </visual>
+    <collision>
+      <geometry>
+        <cylinder radius="0.0275" length="0.28"/>
+      </geometry>
+    </collision>
+    <inertial>
+      <mass value="1.2"/>
+      <inertia ixx="0.012" ixy="0.0" ixz="0.0" iyy="0.012" iyz="0.0" izz="0.012"/>
+    </inertial>
+  </link>
+  <joint name="right_shoulder_joint" type="revolute">
+    <parent link="torso"/>
+    <child link="right_arm_upper"/>
+    <axis xyz="0 1 0"/>
+    <xacro:joint_properties/>
+    <origin xyz="0.16 0 0.38" rpy="0 0 0"/>
+  </joint>
+  <link name="right_arm_elbow">
+    <visual>
+      <geometry>
+        <cylinder radius="0.0225" length="0.04"/>
+      </geometry>
+      <material name="joint_material"/>
+    </visual>
+    <collision>
+      <geometry>
+        <cylinder radius="0.0225" length="0.04"/>
+      </geometry>
+    </collision>
+    <inertial>
+      <mass value="0.3"/>
+      <inertia ixx="0.003" ixy="0.0" ixz="0.0" iyy="0.003" iyz="0.0" izz="0.003"/>
+    </inertial>
+  </link>
+  <joint name="right_elbow_joint" type="revolute">
+    <parent link="right_arm_upper"/>
+    <child link="right_arm_elbow"/>
+    <axis xyz="0 1 0"/>
+    <xacro:joint_properties/>
+    <origin xyz="0 0 0.14" rpy="0 0 0"/>
+  </joint>
+  <link name="right_arm_forearm">
+    <visual>
+      <geometry>
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