Commit message: CORI's URDF has been successfully added to the enviornment and now has a rigidbody + gravity applied.

File: cori_ws/src/cori_description/urdf/cori.urdf.xacro (robot description, xacro)
@@ -1,540 +1,614 @@
 <?xml version="1.0"?>
-<robot name="cori" xmlns:xacro="http://www.ros.org/wiki/xacro">
-<!-- Materials -->
-<material name="body_material">
-  <color rgba="0.82 0.81 0.78 1.0"/> <!-- Light gray for body -->
-</material>
-<material name="joint_material">
-  <color rgba="0.35 0.35 0.35 1.0"/> <!-- Dark gray for joints -->
-</material>
-<material name="screen_material">
-  <color rgba="0.05 0.05 0.05 1.0"/> <!-- Black for screen -->
-</material>
-<material name="eye_material">
-  <color rgba="1.0 1.0 1.0 1.0"/> <!-- White for eyes -->
-</material>
-<!-- Joint Properties Macro -->
-<xacro:macro name="joint_properties">
-  <limit lower="-2.09" upper="2.09" effort="100.0" velocity="1.0"/>
-  <dynamics damping="0.7" friction="0.9"/>
-</xacro:macro>
-<!-- Base Link -->
-<link name="base_link">
-  <visual>
-    <geometry>
-      <cylinder radius="0.05" length="0.02"/>
-    </geometry>
-    <material name="joint_material"/>
-  </visual>
-  <collision>
-    <geometry>
-      <cylinder radius="0.05" length="0.02"/>
-    </geometry>
-  </collision>
-  <inertial>
-    <mass value="0.1"/>
-    <inertia ixx="0.001" ixy="0.0" ixz="0.0" iyy="0.001" iyz="0.0" izz="0.001"/>
-  </inertial>
-</link>
-<!-- Full Body Collision Link - FIXED -->
-<link name="full_body_collision">
-  <collision>
-    <geometry>
-      <box size="0.4 0.3 1.5"/>
-    </geometry>
-  </collision>
-  <inertial>
-    <mass value="5.0"/>
-    <inertia ixx="0.1" ixy="0.0" ixz="0.0" iyy="0.1" iyz="0.0" izz="0.1"/>
-  </inertial>
-</link>
-<joint name="body_collision_joint" type="fixed">
-  <parent link="base_link"/>
-  <child link="full_body_collision"/>
-  <origin xyz="0 0 0" rpy="0 0 0"/>
-</joint>
-<!-- Head Assembly -->
-<link name="head">
-  <visual>
-    <geometry>
-      <box size="0.28 0.2 0.14"/>
-    </geometry>
-    <material name="body_material"/>
-  </visual>
-  <!-- Removed individual collision - using full body STL instead -->
-  <inertial>
-    <mass value="1.5"/>
-    <inertia ixx="0.015" ixy="0.0" ixz="0.0" iyy="0.015" iyz="0.0" izz="0.015"/>
-  </inertial>
-</link>
-<joint name="neck_joint" type="revolute">
-  <parent link="base_link"/>
-  <child link="head"/>
-  <axis xyz="0 0 1"/>
-  <xacro:joint_properties/>
-  <origin xyz="0 0 0.38" rpy="0 0 0"/>
-</joint>
-<link name="screen">
-  <visual>
-    <geometry>
-      <box size="0.22 0.01 0.12"/>
-    </geometry>
-    <material name="screen_material"/>
-  </visual>
-  <inertial>
-    <mass value="0.1"/>
-    <inertia ixx="0.001" ixy="0.0" ixz="0.0" iyy="0.001" iyz="0.0" izz="0.001"/>
-  </inertial>
-</link>
-<joint name="screen_joint" type="fixed">
-  <parent link="head"/>
-  <child link="screen"/>
-  <origin xyz="0 0.1 0.02" rpy="0 0 0"/>
-</joint>
-<link name="left_eye">
-  <visual>
-    <geometry>
-      <sphere radius="0.015"/>
-    </geometry>
-    <material name="eye_material"/>
-  </visual>
-  <inertial>
-    <mass value="0.01"/>
-    <inertia ixx="0.0001" ixy="0.0" ixz="0.0" iyy="0.0001" iyz="0.0" izz="0.0001"/>
-  </inertial>
-</link>
-<joint name="left_eye_joint" type="fixed">
-  <parent link="screen"/>
-  <child link="left_eye"/>
-  <origin xyz="-0.08 0.02 0.02" rpy="0 0 0"/>
-</joint>
-<link name="right_eye">
-  <visual>
-    <geometry>
-      <sphere radius="0.015"/>
-    </geometry>
-    <material name="eye_material"/>
-  </visual>
-  <inertial>
-    <mass value="0.01"/>
-    <inertia ixx="0.0001" ixy="0.0" ixz="0.0" iyy="0.0001" iyz="0.0" izz="0.0001"/>
-  </inertial>
-</link>
-<joint name="right_eye_joint" type="fixed">
-  <parent link="screen"/>
-  <child link="right_eye"/>
-  <origin xyz="0.08 0.02 0.02" rpy="0 0 0"/>
-</joint>
-<!-- Torso Assembly -->
-<link name="torso">
-  <visual>
-    <geometry>
-      <box size="0.32 0.22 0.38"/>
-    </geometry>
-    <material name="body_material"/>
-  </visual>
-  <!-- Removed individual collision - using full body STL instead -->
-  <inertial>
-    <mass value="8.0"/>
-    <inertia ixx="0.08" ixy="0.0" ixz="0.0" iyy="0.08" iyz="0.0" izz="0.08"/>
-  </inertial>
-</link>
-<joint name="waist_joint" type="revolute">
-  <parent link="base_link"/>
-  <child link="torso"/>
-  <axis xyz="0 0 1"/>
-  <xacro:joint_properties/>
-  <origin xyz="0 0 0" rpy="0 0 0"/>
-</joint>
-<!-- Finger Macro -->
-<xacro:macro name="finger" params="hand name offset">
-  <link name="${hand}_finger_${name}">
-    <visual>
-      <geometry>
-        <cylinder radius="0.006" length="0.06"/>
-      </geometry>
-      <material name="joint_material"/>
+<robot xmlns:xacro="http://www.ros.org/wiki/xacro" name="cori">
+  <!-- Materials -->
+  <material name="body_material">
+    <color rgba="0.82 0.81 0.78 1.0"/> <!-- Light gray for body -->
+  </material>
+  <material name="joint_material">
+    <color rgba="0.35 0.35 0.35 1.0"/> <!-- Dark gray for joints -->
+  </material>
+  <material name="screen_material">
+    <color rgba="0.05 0.05 0.05 1.0"/> <!-- Black for screen -->
+  </material>
+  <material name="eye_material">
+    <color rgba="1.0 1.0 1.0 1.0"/> <!-- White for eyes -->
+  </material>
+  <material name="invisible">
+    <color rgba="0.0 0.0 0.0 0.0"/> <!-- Transparent -->
+  </material>
+  <!-- Base Link -->
+  <link name="base_link">
+    <visual>
+      <geometry>
+        <cylinder radius="0.15" length="0.05"/>
+      </geometry>
+      <material name="invisible"/> <!-- Make base invisible -->
     </visual>
     <collision>
       <geometry>
-        <cylinder radius="0.006" length="0.06"/>
+        <cylinder radius="0.15" length="0.05"/>
       </geometry>
     </collision>
     <inertial>
+      <mass value="1.0"/>
+      <inertia ixx="0.01" ixy="0.0" ixz="0.0" iyy="0.01" iyz="0.0" izz="0.01"/>
+    </inertial>
+  </link>
+  <!-- Full Body Collision Link - THIS WILL SHOW YOUR STL MESH -->
+  <link name="full_body_collision">
+    <visual>
+      <geometry>
+        <mesh filename="file:///home/juptegraph/Workspaces/Robotics/Projects/CORI/cori_ws/src/cori_description/meshes/CORI_Solid.stl" scale="0.03 0.03 0.03"/>
+      </geometry>
+      <material name="body_material"/>
+    </visual>
+    <collision>
+      <geometry>
+        <mesh filename="file:///home/juptegraph/Workspaces/Robotics/Projects/CORI/cori_ws/src/cori_description/meshes/CORI_Solid.stl" scale="0.03 0.03 0.03"/>
+      </geometry>
+    </collision>
+    <inertial>
+      <mass value="50.0"/>
+      <inertia ixx="2.0" ixy="0.0" ixz="0.0" iyy="2.0" iyz="0.0" izz="1.0"/>
+    </inertial>
+  </link>
+  <!-- Joint connecting base to full body -->
+  <joint name="base_to_body" type="fixed">
+    <parent link="base_link"/>
+    <child link="full_body_collision"/>
+    <origin xyz="-0.07 0 0.025" rpy="0 0 1.57"/>
+  </joint>
+  <!-- Torso - Made invisible -->
+  <link name="torso">
+    <visual>
+      <geometry>
+        <cylinder radius="0.12" length="0.25"/>
+      </geometry>
+      <material name="invisible"/>
+    </visual>
+    <inertial>
+      <mass value="5.0"/>
+      <inertia ixx="0.05" ixy="0.0" ixz="0.0" iyy="0.05" iyz="0.0" izz="0.02"/>
+    </inertial>
+  </link>
+  <joint name="body_to_torso" type="fixed">
+    <parent link="full_body_collision"/>
+    <child link="torso"/>
+    <origin xyz="0 0 0.125" rpy="0 0 0"/>
+  </joint>
+  <!-- Head - Made invisible -->
+  <link name="head">
+    <visual>
+      <geometry>
+        <sphere radius="0.08"/>
+      </geometry>
+      <material name="invisible"/>
+    </visual>
+    <inertial>
+      <mass value="1.0"/>
+      <inertia ixx="0.01" ixy="0.0" ixz="0.0" iyy="0.01" iyz="0.0" izz="0.01"/>
+    </inertial>
+  </link>
+  <joint name="torso_to_head" type="revolute">
+    <parent link="torso"/>
+    <child link="head"/>
+    <origin xyz="0 0 0.15" rpy="0 0 0"/>
+    <axis xyz="0 0 1"/>
+    <limit lower="-1.57" upper="1.57" effort="10" velocity="1"/>
+  </joint>
+  <!-- Screen - Made invisible -->
+  <link name="screen">
+    <visual>
+      <geometry>
+        <box size="0.05 0.03 0.01"/>
+      </geometry>
+      <material name="invisible"/>
+    </visual>
+    <inertial>
       <mass value="0.1"/>
-      <inertia ixx="0.0001" ixy="0.0" ixz="0.0" iyy="0.0001" iyz="0.0" izz="0.0001"/>
-    </inertial>
-  </link>
-  <joint name="${hand}_finger_${name}_joint" type="revolute">
-    <parent link="${hand}_hand_palm"/>
-    <child link="${hand}_finger_${name}"/>
+      <inertia ixx="0.001" ixy="0.0" ixz="0.0" iyy="0.001" iyz="0.0" izz="0.001"/>
+    </inertial>
+  </link>
+  <joint name="head_to_screen" type="fixed">
+    <parent link="head"/>
+    <child link="screen"/>
+    <origin xyz="0.07 0 0" rpy="0 0 0"/>
+  </joint>
+  <!-- Eyes - Made invisible -->
+  <link name="left_eye">
+    <visual>
+      <geometry>
+        <sphere radius="0.01"/>
+      </geometry>
+      <material name="invisible"/>
+    </visual>
+    <inertial>
+      <mass value="0.01"/>
+      <inertia ixx="0.0001" ixy="0.0" ixz="0.0" iyy="0.0001" iyz="0.0" izz="0.0001"/>
+    </inertial>
+  </link>
+  <joint name="head_to_left_eye" type="fixed">
+    <parent link="head"/>
+    <child link="left_eye"/>
+    <origin xyz="0.06 0.02 0.02" rpy="0 0 0"/>
+  </joint>
+  <link name="right_eye">
+    <visual>
+      <geometry>
+        <sphere radius="0.01"/>
+      </geometry>
+      <material name="invisible"/>
+    </visual>
+    <inertial>
+      <mass value="0.01"/>
+      <inertia ixx="0.0001" ixy="0.0" ixz="0.0" iyy="0.0001" iyz="0.0" izz="0.0001"/>
+    </inertial>
+  </link>
+  <joint name="head_to_right_eye" type="fixed">
+    <parent link="head"/>
+    <child link="right_eye"/>
+    <origin xyz="0.06 -0.02 0.02" rpy="0 0 0"/>
+  </joint>
+  <!-- Left Arm Chain - Made invisible -->
+  <link name="left_arm_upper">
+    <visual>
+      <geometry>
+        <cylinder radius="0.03" length="0.15"/>
+      </geometry>
+      <material name="invisible"/>
+    </visual>
+    <inertial>
+      <mass value="1.0"/>
+      <inertia ixx="0.01" ixy="0.0" ixz="0.0" iyy="0.01" iyz="0.0" izz="0.001"/>
+    </inertial>
+  </link>
+  <joint name="torso_to_left_arm" type="revolute">
+    <parent link="torso"/>
+    <child link="left_arm_upper"/>
+    <origin xyz="0 0.14 0.1" rpy="1.57 0 6.28"/>
+    <axis xyz="1 0 0"/>
+    <limit lower="-3.14" upper="3.14" effort="10" velocity="1"/>
+  </joint>
+  <link name="left_arm_elbow">
+    <visual>
+      <geometry>
+        <sphere radius="0.025"/>
+      </geometry>
+      <material name="invisible"/>
+    </visual>
+    <inertial>
+      <mass value="0.2"/>
+      <inertia ixx="0.001" ixy="0.0" ixz="0.0" iyy="0.001" iyz="0.0" izz="0.001"/>
+    </inertial>
+  </link>
+  <joint name="left_arm_to_elbow" type="revolute">
+    <parent link="left_arm_upper"/>
+    <child link="left_arm_elbow"/>
+    <origin xyz="0 0 0.075" rpy="0 0 0"/>
+    <axis xyz="1 0 0"/>
+    <limit lower="-2.0" upper="2.0" effort="10" velocity="1"/>
+  </joint>
+  <link name="left_arm_forearm">
+    <visual>
+      <geometry>
+        <cylinder radius="0.025" length="0.12"/>
+      </geometry>
+      <material name="invisible"/>
+    </visual>
+    <inertial>
+      <mass value="0.8"/>
+      <inertia ixx="0.008" ixy="0.0" ixz="0.0" iyy="0.008" iyz="0.0" izz="0.001"/>
+    </inertial>
+  </link>
+  <joint name="left_elbow_to_forearm" type="revolute">
+    <parent link="left_arm_elbow"/>
+    <child link="left_arm_forearm"/>
+    <origin xyz="0 0 0.06" rpy="0 0 0"/>
+    <axis xyz="1 0 0"/>
+    <limit lower="-1.5" upper="1.5" effort="10" velocity="1"/>
+  </joint>
+  <link name="left_hand_palm">
+    <visual>
+      <geometry>
+        <box size="0.06 0.04 0.02"/>
+      </geometry>
+      <material name="invisible"/>
+    </visual>
+    <inertial>
+      <mass value="0.3"/>
+      <inertia ixx="0.001" ixy="0.0" ixz="0.0" iyy="0.001" iyz="0.0" izz="0.001"/>
+    </inertial>
+  </link>
+  <joint name="left_forearm_to_hand" type="revolute">
+    <parent link="left_arm_forearm"/>
+    <child link="left_hand_palm"/>
+    <origin xyz="0 0 0.08" rpy="0 0 0"/>
     <axis xyz="0 0 1"/>
-    <limit lower="0.0" upper="1.57" effort="50.0" velocity="0.5"/>
-    <dynamics damping="0.5" friction="0.7"/>
-    <origin xyz="${offset} 0 -0.025" rpy="0 0 0"/>
-  </joint>
-</xacro:macro>
-<!-- Left Arm -->
-<link name="left_arm_upper">
-  <visual>
-    <geometry>
-      <cylinder radius="0.0275" length="0.28"/>
-    </geometry>
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
Commit message: Migrated CORI filepaths from absolute to relative.

File: cori_ws/src/cori_description/urdf/cori.urdf.xacro (robot description, xacro)
@@ -23,5 +23,5 @@
       <origin xyz="0 0 0" rpy="0 0 0"/>
       <geometry>
-        <mesh filename="file:///home/juptegraph/Workspaces/Robotics/Projects/CORI/cori_ws/src/cori_description/meshes/cori_body_v1.0/cori_torso.stl" scale="0.35 0.35 0.35"/>
+        <mesh filename="package://cori_description/meshes/cori_body_v1.0/cori_torso.stl" scale="0.35 0.35 0.35"/>
       </geometry>
       <material name="cori_white"/>
@@ -47,5 +47,5 @@
       <origin xyz="0 0 0" rpy="0 0 0"/>
       <geometry>
-        <mesh filename="file:///home/juptegraph/Workspaces/Robotics/Projects/CORI/cori_ws/src/cori_description/meshes/cori_body_v1.0/cori_head.stl" scale="0.35 0.35 0.35"/>
+        <mesh filename="package://cori_description/meshes/cori_body_v1.0/cori_head.stl" scale="0.35 0.35 0.35"/>
       </geometry>
       <material name="cori_head"/>
@@ -74,5 +74,5 @@
       <origin xyz="0 0 0" rpy="0 0 0"/>
       <geometry>
-        <mesh filename="file:///home/juptegraph/Workspaces/Robotics/Projects/CORI/cori_ws/src/cori_description/meshes/cori_body_v1.0/cori_pelvis.stl" scale="0.35 0.35 0.35"/>
+        <mesh filename="package://cori_description/meshes/cori_body_v1.0/cori_pelvis.stl" scale="0.35 0.35 0.35"/>
       </geometry>
       <material name="cori_white"/>
@@ -98,5 +98,5 @@
       <origin xyz="0 0 0" rpy="0 0 0"/>
       <geometry>
-        <mesh filename="file:///home/juptegraph/Workspaces/Robotics/Projects/CORI/cori_ws/src/cori_description/meshes/cori_body_v1.0/cori_left_upper_arm.stl" scale="0.35 0.35 0.35"/>
+        <mesh filename="package://cori_description/meshes/cori_body_v1.0/cori_left_upper_arm.stl" scale="0.35 0.35 0.35"/>
       </geometry>
       <material name="cori_white"/>
@@ -125,5 +125,5 @@
       <origin xyz="0 0 0" rpy="0 0 0"/>
       <geometry>
-        <mesh filename="file:///home/juptegraph/Workspaces/Robotics/Projects/CORI/cori_ws/src/cori_description/meshes/cori_body_v1.0/cori_left_forearm.stl" scale="0.35 0.35 0.35"/>
+        <mesh filename="package://cori_description/meshes/cori_body_v1.0/cori_left_forearm.stl" scale="0.35 0.35 0.35"/>
       </geometry>
       <material name="cori_white"/>
@@ -152,5 +152,5 @@
       <origin xyz="0 0 0" rpy="0 0 0"/>
       <geometry>
-        <mesh filename="file:///home/juptegraph/Workspaces/Robotics/Projects/CORI/cori_ws/src/cori_description/meshes/cori_body_v1.0/cori_left_hand.stl" scale="0.35 0.35 0.35"/>
+        <mesh filename="package://cori_description/meshes/cori_body_v1.0/cori_left_hand.stl" scale="0.35 0.35 0.35"/>
       </geometry>
       <material name="cori_white"/>
@@ -179,5 +179,5 @@
       <origin xyz="0 0 0" rpy="0 0 0"/>
       <geometry>
-        <mesh filename="file:///home/juptegraph/Workspaces/Robotics/Projects/CORI/cori_ws/src/cori_description/meshes/cori_body_v1.0/cori_right_upper_arm.stl" scale="0.35 0.35 0.35"/>
+        <mesh filename="package://cori_description/meshes/cori_body_v1.0/cori_right_upper_arm.stl" scale="0.35 0.35 0.35"/>
       </geometry>
       <material name="cori_white"/>
@@ -206,5 +206,5 @@
       <origin xyz="0 0 0" rpy="0 0 0"/>
       <geometry>
-        <mesh filename="file:///home/juptegraph/Workspaces/Robotics/Projects/CORI/cori_ws/src/cori_description/meshes/cori_body_v1.0/cori_right_forearm.stl" scale="0.35 0.35 0.35"/>
+        <mesh filename="package://cori_description/meshes/cori_body_v1.0/cori_right_forearm.stl" scale="0.35 0.35 0.35"/>
       </geometry>
       <material name="cori_white"/>
@@ -233,5 +233,5 @@
       <origin xyz="0 0 0" rpy="0 0 0"/>
       <geometry>
-        <mesh filename="file:///home/juptegraph/Workspaces/Robotics/Projects/CORI/cori_ws/src/cori_description/meshes/cori_body_v1.0/cori_right_hand.stl" scale="0.35 0.35 0.35"/>
+        <mesh filename="package://cori_description/meshes/cori_body_v1.0/cori_right_hand.stl" scale="0.35 0.35 0.35"/>
       </geometry>
       <material name="cori_white"/>
@@ -260,5 +260,5 @@
       <origin xyz="0 0 0" rpy="0 0 0"/>
       <geometry>
-        <mesh filename="file:///home/juptegraph/Workspaces/Robotics/Projects/CORI/cori_ws/src/cori_description/meshes/cori_body_v1.0/cori_left_thigh.stl" scale="0.35 0.35 0.35"/>
+        <mesh filename="package://cori_description/meshes/cori_body_v1.0/cori_left_thigh.stl" scale="0.35 0.35 0.35"/>
       </geometry>
       <material name="cori_white"/>
@@ -287,5 +287,5 @@
       <origin xyz="0 0 0" rpy="0 0 0"/>
       <geometry>
-        <mesh filename="file:///home/juptegraph/Workspaces/Robotics/Projects/CORI/cori_ws/src/cori_description/meshes/cori_body_v1.0/cori_left_shin.stl" scale="0.35 0.35 0.35"/>
+        <mesh filename="package://cori_description/meshes/cori_body_v1.0/cori_left_shin.stl" scale="0.35 0.35 0.35"/>
       </geometry>
       <material name="cori_white"/>
@@ -314,5 +314,5 @@
       <origin xyz="0 0 0" rpy="0 0 0"/>
       <geometry>
-        <mesh filename="file:///home/juptegraph/Workspaces/Robotics/Projects/CORI/cori_ws/src/cori_description/meshes/cori_body_v1.0/cori_left_knee.stl" scale="0.35 0.35 0.35"/>
+        <mesh filename="package://cori_description/meshes/cori_body_v1.0/cori_left_knee.stl" scale="0.35 0.35 0.35"/>
       </geometry>
       <material name="cori_white"/>
@@ -338,5 +338,5 @@
       <origin xyz="0 0 0" rpy="0 0 0"/>
       <geometry>
-        <mesh filename="file:///home/juptegraph/Workspaces/Robotics/Projects/CORI/cori_ws/src/cori_description/meshes/cori_body_v1.0/cori_left_foot.stl" scale="0.35 0.35 0.35"/>
+        <mesh filename="package://cori_description/meshes/cori_body_v1.0/cori_left_foot.stl" scale="0.35 0.35 0.35"/>
       </geometry>
       <material name="cori_white"/>
@@ -365,5 +365,5 @@
       <origin xyz="0 0 0" rpy="0 0 0"/>
       <geometry>
-        <mesh filename="file:///home/juptegraph/Workspaces/Robotics/Projects/CORI/cori_ws/src/cori_description/meshes/cori_body_v1.0/cori_right_thigh.stl" scale="0.35 0.35 0.35"/>
+        <mesh filename="package://cori_description/meshes/cori_body_v1.0/cori_right_thigh.stl" scale="0.35 0.35 0.35"/>
       </geometry>
       <material name="cori_white"/>
@@ -392,5 +392,5 @@
       <origin xyz="0 0 0" rpy="0 0 0"/>
       <geometry>
-        <mesh filename="file:///home/juptegraph/Workspaces/Robotics/Projects/CORI/cori_ws/src/cori_description/meshes/cori_body_v1.0/cori_right_shin.stl" scale="0.35 0.35 0.35"/>
+        <mesh filename="package://cori_description/meshes/cori_body_v1.0/cori_right_shin.stl" scale="0.35 0.35 0.35"/>
       </geometry>
       <material name="cori_white"/>
@@ -419,5 +419,5 @@
       <origin xyz="0 0 0" rpy="0 0 0"/>
       <geometry>
-        <mesh filename="file:///home/juptegraph/Workspaces/Robotics/Projects/CORI/cori_ws/src/cori_description/meshes/cori_body_v1.0/cori_right_knee.stl" scale="0.35 0.35 0.35"/>
+        <mesh filename="package://cori_description/meshes/cori_body_v1.0/cori_right_knee.stl" scale="0.35 0.35 0.35"/>
       </geometry>
       <material name="cori_white"/>
@@ -443,5 +443,5 @@
       <origin xyz="0 0 0" rpy="0 0 0"/>
       <geometry>
-        <mesh filename="file:///home/juptegraph/Workspaces/Robotics/Projects/CORI/cori_ws/src/cori_description/meshes/cori_body_v1.0/cori_right_foot.stl" scale="0.35 0.35 0.35"/>
+        <mesh filename="package://cori_description/meshes/cori_body_v1.0/cori_right_foot.stl" scale="0.35 0.35 0.35"/>
       </geometry>
       <material name="cori_white"/>
