Commit message: Menu & nav system changes, close to full camera detection and gazebo head adjustment with real feedback & adjustment.

File: cori_ws/src/cori_description/urdf/cori.urdf.xacro (robot description, xacro)
@@ -23,5 +23,5 @@
       <origin xyz="0 0 0" rpy="0 0 0"/>
       <geometry>
-        <mesh filename="package://cori_description/meshes/cori_body_v1.0/cori_torso.stl" scale="0.35 0.35 0.35"/>
+        <mesh filename="file:///home/juptegraph/Workspaces/Robotics/Projects/CORI/cori_ws/src/cori_description/meshes/cori_body_v1.0/cori_torso.stl" scale="0.35 0.35 0.35"/>
       </geometry>
       <material name="cori_white"/>
@@ -47,5 +47,5 @@
       <origin xyz="0 0 0" rpy="0 0 0"/>
       <geometry>
-        <mesh filename="package://cori_description/meshes/cori_body_v1.0/cori_head.stl" scale="0.35 0.35 0.35"/>
+        <mesh filename="file:///home/juptegraph/Workspaces/Robotics/Projects/CORI/cori_ws/src/cori_description/meshes/cori_body_v1.0/cori_head.stl" scale="0.35 0.35 0.35"/>
       </geometry>
       <material name="cori_head"/>
@@ -74,5 +74,5 @@
       <origin xyz="0 0 0" rpy="0 0 0"/>
       <geometry>
-        <mesh filename="package://cori_description/meshes/cori_body_v1.0/cori_pelvis.stl" scale="0.35 0.35 0.35"/>
+        <mesh filename="file:///home/juptegraph/Workspaces/Robotics/Projects/CORI/cori_ws/src/cori_description/meshes/cori_body_v1.0/cori_pelvis.stl" scale="0.35 0.35 0.35"/>
       </geometry>
       <material name="cori_white"/>
@@ -98,5 +98,5 @@
       <origin xyz="0 0 0" rpy="0 0 0"/>
       <geometry>
-        <mesh filename="package://cori_description/meshes/cori_body_v1.0/cori_left_upper_arm.stl" scale="0.35 0.35 0.35"/>
+        <mesh filename="file:///home/juptegraph/Workspaces/Robotics/Projects/CORI/cori_ws/src/cori_description/meshes/cori_body_v1.0/cori_left_upper_arm.stl" scale="0.35 0.35 0.35"/>
       </geometry>
       <material name="cori_white"/>
@@ -125,5 +125,5 @@
       <origin xyz="0 0 0" rpy="0 0 0"/>
       <geometry>
-        <mesh filename="package://cori_description/meshes/cori_body_v1.0/cori_left_forearm.stl" scale="0.35 0.35 0.35"/>
+        <mesh filename="file:///home/juptegraph/Workspaces/Robotics/Projects/CORI/cori_ws/src/cori_description/meshes/cori_body_v1.0/cori_left_forearm.stl" scale="0.35 0.35 0.35"/>
       </geometry>
       <material name="cori_white"/>
@@ -152,5 +152,5 @@
       <origin xyz="0 0 0" rpy="0 0 0"/>
       <geometry>
-        <mesh filename="package://cori_description/meshes/cori_body_v1.0/cori_left_hand.stl" scale="0.35 0.35 0.35"/>
+        <mesh filename="file:///home/juptegraph/Workspaces/Robotics/Projects/CORI/cori_ws/src/cori_description/meshes/cori_body_v1.0/cori_left_hand.stl" scale="0.35 0.35 0.35"/>
       </geometry>
       <material name="cori_white"/>
@@ -179,5 +179,5 @@
       <origin xyz="0 0 0" rpy="0 0 0"/>
       <geometry>
-        <mesh filename="package://cori_description/meshes/cori_body_v1.0/cori_right_upper_arm.stl" scale="0.35 0.35 0.35"/>
+        <mesh filename="file:///home/juptegraph/Workspaces/Robotics/Projects/CORI/cori_ws/src/cori_description/meshes/cori_body_v1.0/cori_right_upper_arm.stl" scale="0.35 0.35 0.35"/>
       </geometry>
       <material name="cori_white"/>
@@ -206,5 +206,5 @@
       <origin xyz="0 0 0" rpy="0 0 0"/>
       <geometry>
-        <mesh filename="package://cori_description/meshes/cori_body_v1.0/cori_right_forearm.stl" scale="0.35 0.35 0.35"/>
+        <mesh filename="file:///home/juptegraph/Workspaces/Robotics/Projects/CORI/cori_ws/src/cori_description/meshes/cori_body_v1.0/cori_right_forearm.stl" scale="0.35 0.35 0.35"/>
       </geometry>
       <material name="cori_white"/>
@@ -233,5 +233,5 @@
       <origin xyz="0 0 0" rpy="0 0 0"/>
       <geometry>
-        <mesh filename="package://cori_description/meshes/cori_body_v1.0/cori_right_hand.stl" scale="0.35 0.35 0.35"/>
+        <mesh filename="file:///home/juptegraph/Workspaces/Robotics/Projects/CORI/cori_ws/src/cori_description/meshes/cori_body_v1.0/cori_right_hand.stl" scale="0.35 0.35 0.35"/>
       </geometry>
       <material name="cori_white"/>
@@ -260,5 +260,5 @@
       <origin xyz="0 0 0" rpy="0 0 0"/>
       <geometry>
-        <mesh filename="package://cori_description/meshes/cori_body_v1.0/cori_left_thigh.stl" scale="0.35 0.35 0.35"/>
+        <mesh filename="file:///home/juptegraph/Workspaces/Robotics/Projects/CORI/cori_ws/src/cori_description/meshes/cori_body_v1.0/cori_left_thigh.stl" scale="0.35 0.35 0.35"/>
       </geometry>
       <material name="cori_white"/>
@@ -287,5 +287,5 @@
       <origin xyz="0 0 0" rpy="0 0 0"/>
       <geometry>
-        <mesh filename="package://cori_description/meshes/cori_body_v1.0/cori_left_shin.stl" scale="0.35 0.35 0.35"/>
+        <mesh filename="file:///home/juptegraph/Workspaces/Robotics/Projects/CORI/cori_ws/src/cori_description/meshes/cori_body_v1.0/cori_left_shin.stl" scale="0.35 0.35 0.35"/>
       </geometry>
       <material name="cori_white"/>
@@ -314,5 +314,5 @@
       <origin xyz="0 0 0" rpy="0 0 0"/>
       <geometry>
-        <mesh filename="package://cori_description/meshes/cori_body_v1.0/cori_left_knee.stl" scale="0.35 0.35 0.35"/>
+        <mesh filename="file:///home/juptegraph/Workspaces/Robotics/Projects/CORI/cori_ws/src/cori_description/meshes/cori_body_v1.0/cori_left_knee.stl" scale="0.35 0.35 0.35"/>
       </geometry>
       <material name="cori_white"/>
@@ -338,5 +338,5 @@
       <origin xyz="0 0 0" rpy="0 0 0"/>
       <geometry>
-        <mesh filename="package://cori_description/meshes/cori_body_v1.0/cori_left_foot.stl" scale="0.35 0.35 0.35"/>
+        <mesh filename="file:///home/juptegraph/Workspaces/Robotics/Projects/CORI/cori_ws/src/cori_description/meshes/cori_body_v1.0/cori_left_foot.stl" scale="0.35 0.35 0.35"/>
       </geometry>
       <material name="cori_white"/>
@@ -365,5 +365,5 @@
       <origin xyz="0 0 0" rpy="0 0 0"/>
       <geometry>
-        <mesh filename="package://cori_description/meshes/cori_body_v1.0/cori_right_thigh.stl" scale="0.35 0.35 0.35"/>
+        <mesh filename="file:///home/juptegraph/Workspaces/Robotics/Projects/CORI/cori_ws/src/cori_description/meshes/cori_body_v1.0/cori_right_thigh.stl" scale="0.35 0.35 0.35"/>
       </geometry>
       <material name="cori_white"/>
@@ -392,5 +392,5 @@
       <origin xyz="0 0 0" rpy="0 0 0"/>
       <geometry>
-        <mesh filename="package://cori_description/meshes/cori_body_v1.0/cori_right_shin.stl" scale="0.35 0.35 0.35"/>
+        <mesh filename="file:///home/juptegraph/Workspaces/Robotics/Projects/CORI/cori_ws/src/cori_description/meshes/cori_body_v1.0/cori_right_shin.stl" scale="0.35 0.35 0.35"/>
       </geometry>
       <material name="cori_white"/>
@@ -419,5 +419,5 @@
       <origin xyz="0 0 0" rpy="0 0 0"/>
       <geometry>
-        <mesh filename="package://cori_description/meshes/cori_body_v1.0/cori_right_knee.stl" scale="0.35 0.35 0.35"/>
+        <mesh filename="file:///home/juptegraph/Workspaces/Robotics/Projects/CORI/cori_ws/src/cori_description/meshes/cori_body_v1.0/cori_right_knee.stl" scale="0.35 0.35 0.35"/>
       </geometry>
       <material name="cori_white"/>
@@ -443,5 +443,5 @@
       <origin xyz="0 0 0" rpy="0 0 0"/>
       <geometry>
-        <mesh filename="package://cori_description/meshes/cori_body_v1.0/cori_right_foot.stl" scale="0.35 0.35 0.35"/>
+        <mesh filename="file:///home/juptegraph/Workspaces/Robotics/Projects/CORI/cori_ws/src/cori_description/meshes/cori_body_v1.0/cori_right_foot.stl" scale="0.35 0.35 0.35"/>
       </geometry>
       <material name="cori_white"/>
